File: pcb/main_MagicAlonso/CH340G_programmer.kicad_sch (KiCad schematic)
At the start: 8 parts, among them J11 USB_B_Micro, J2 Conn_01x05_Pin, J3 Conn_01x04_Pin, U4 CH340C

Commit message: more schematic
Parts:
- added J4: USB_C_Receptacle_USB2.0_16P, symbol Connector:USB_C_Receptacle_USB2.0_16P
Connections:
- new net: J4.A1 (GND), J4.A12 (GND), J4.B1 (GND), J4.B12 (GND)
- new net: J4.A4 (VBUS), J4.A9 (VBUS), J4.B4 (VBUS), J4.B9 (VBUS)
Other:
- moved on the sheet: J2
Changed lines of the file:
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@@
-	)
-	(junction
-		(at 127 43.18)
-		(diameter 0)
-		(color 0 0 0 0)
 	)
 	(junction
@@
 	)
 	(no_connect
-		(at 66.294 89.408)
+		(at 67.31 86.36)
 	)
 	(no_connect
@@
 	(wire
 		(pts
+			(xy 127 40.64) (xy 127 44.45)
+		)
+		(stroke
+			(width 0)
+			(type default)
+		)
+	)
+	(wire
+		(pts
 			(xy 204.47 41.91) (xy 210.82 41.91)
 		)
@@
 	(wire
 		(pts
-			(xy 124.46 44.45) (xy 124.46 43.18)
+			(xy 124.46 44.45) (xy 124.46 40.64)
 		)
 		(stroke
@@
 	(wire
 		(pts
-			(xy 65.024 81.788) (xy 66.294 81.788)
+			(xy 66.04 78.74) (xy 67.31 78.74)
 		)
 		(stroke
@@
 	(wire
 		(pts
-			(xy 66.294 91.948) (xy 57.404 91.948)
-		)
-		(stroke
-			(width 0)
-			(type default)
-		)
-	)
-	(wire
-		(pts
-			(xy 65.024 84.328) (xy 66.294 84.328)
-		)
-		(stroke
-			(width 0)
-			(type default)
-		)
-	)
-	(wire
-		(pts
-			(xy 127 40.64) (xy 127 43.18)
+			(xy 67.31 88.9) (xy 58.42 88.9)
+		)
+		(stroke
+			(width 0)
+			(type default)
+		)
+	)
+	(wire
+		(pts
+			(xy 66.04 81.28) (xy 67.31 81.28)
 		)
 		(stroke
@@
 	(wire
 		(pts
-			(xy 57.404 91.948) (xy 57.404 93.218)
+			(xy 58.42 88.9) (xy 58.42 90.17)
 		)
 		(stroke
@@
 	(wire
 		(pts
-			(xy 65.024 86.868) (xy 66.294 86.868)
+			(xy 66.04 83.82) (xy 67.31 83.82)
 		)
 		(stroke
@@
 	(wire
 		(pts
-			(xy 124.46 43.18) (xy 127 43.18)
+			(xy 124.46 40.64) (xy 127 40.64)
 		)
 		(stroke
@@
 		(pts
 			(xy 210.82 48.26) (xy 210.82 46.99)
-		)
-		(stroke
-			(width 0)
-			(type default)
-		)
-	)
-	(wire
-		(pts
-			(xy 127 43.18) (xy 127 44.45)
 		)
 		(stroke
@@
 	)
 	(label "D+"
-		(at 65.024 86.868 180)
+		(at 66.04 83.82 180)
 		(effects
 			(font
@@
 	)
 	(label "D-"
-		(at 65.024 84.328 180)
+		(at 66.04 81.28 180)
 		(effects
 			(font
@@
 	)
 	(label "Vbus"
-		(at 65.024 81.788 180)
+		(at 66.04 78.74 180)
 		(effects
 			(font
@@
 	(symbol
 		(lib_id "Connector:Conn_01x05_Pin")
-		(at 71.374 86.868 180)
+		(at 72.39 83.82 180)
 		(unit 1)
 		(exclude_from_sim no)
@@
 		(fields_autoplaced yes)
 		(property "Reference" "J2"
-			(at 72.644 85.5979 0)
+			(at 73.66 82.5499 0)
 			(effects
 				(font
@@
 		)
 		(property "Value" "Conn_01x05_Pin"
-			(at 72.644 88.1379 0)
+			(at 73.66 85.0899 0)
 			(effects
 				(font
@@
 		)
 		(property "Footprint" ""
-			(at 71.374 86.868 0)
+			(at 72.39 83.82 0)
 			(effects
 				(font
@@
 		)
 		(property "Datasheet" "~"
-			(at 71.374 86.868 0)
+			(at 72.39 83.82 0)
 			(effects
 				(font
@@
 		)
 		(property "Description" "Generic connector, single row, 01x05, script generated"
-			(at 71.374 86.868 0)
+			(at 72.39 83.82 0)
 			(effects
 				(font
@@
 				(path "/dedd09af-bea2-4be5-843e-bc5c56d4d8f5/82b42807-ad94-4f54-a6bf-1ac7ea765fbf"
 					(reference "#PWR046")
+					(unit 1)
+				)
+			)
+		)
+	)
+	(symbol
+		(lib_id "Connector:USB_C_Receptacle_USB2.0_16P")
+		(at -8.89 60.96 0)
+		(unit 1)
+		(exclude_from_sim no)
+		(in_bom yes)
+		(on_board yes)
+		(dnp no)
+		(fields_autoplaced yes)
+		(property "Reference" "J4"
+			(at -8.89 38.1 0)
+			(effects
+				(font
+					(size 1.27 1.27)
+				)
+			)
+		)
+		(property "Value" "USB_C_Receptacle_USB2.0_16P"
+			(at -8.89 40.64 0)
+			(effects
+				(font
+					(size 1.27 1.27)
+				)
+			)
+		)
+		(property "Footprint" ""
+			(at -5.08 60.96 0)
+			(effects
+				(font
+					(size 1.27 1.27)
+				)
+				(hide yes)
+			)
+		)
+		(property "Datasheet" "https://www.usb.org/sites/default/files/documents/usb_type-c.zip"
+			(at -5.08 60.96 0)
+			(effects
+				(font
+					(size 1.27 1.27)
+				)
+				(hide yes)
+			)
+		)
+		(property "Description" "USB 2.0-only 16P Type-C Receptacle connector"
+			(at -8.89 60.96 0)
+			(effects
+				(font
+					(size 1.27 1.27)
+				)
+				(hide yes)
+			)
+		)
+		(pin "A12"
+		)
+		(pin "A1"
+		)
+		(pin "A5"
+		)
+		(pin "S1"
+		)
+		(pin "B1"
+		)
+		(pin "A4"
+		)
+		(pin "A9"
+		)
+		(pin "B12"
+		)
+		(pin "B4"
+		)
+		(pin "B9"
+		)
+		(pin "A6"
+		)
+		(pin "A8"
+		)
+		(pin "A7"
+		)
+		(pin "B6"
+		)
+		(pin "B7"
+		)
+		(pin "B8"
+		)
+		(pin "B5"
+		)
+		(instances
+			(project "main_MagicAlonso"
+				(path "/80af5e1a-3060-4775-9fc3-f6762d1535e7/c19a4b5e-b66e-4d93-9513-18dbfa3808b4"
+					(reference "J4")
 					(unit 1)
 				)
@@
 	(symbol
 		(lib_id "power:GND")
-		(at 57.404 93.218 0)
+		(at 58.42 90.17 0)
 		(unit 1)
 		(exclude_from_sim no)
@@
 		(dnp no)
 		(property "Reference" "#PWR036"
-			(at 57.404 99.568 0)
+			(at 58.42 96.52 0)
 			(effects
 				(font
@@
 		)
 		(property "Value" "GND"
-			(at 57.404 97.536 0)
+			(at 58.42 94.488 0)
 			(effects
 				(font
@@
 		)
 		(property "Footprint" ""
-			(at 57.404 93.218 0)
+			(at 58.42 90.17 0)
 			(effects
 				(font
@@
 		)
 		(property "Datasheet" ""
-			(at 57.404 93.218 0)
+			(at 58.42 90.17 0)
 			(effects
 				(font
@@
 		)
 		(property "Description" "Power symbol creates a global label with name \"GND\" , ground"
-			(at 57.404 93.218 0)
-			(effects
-				(font
+			(at 58.42 90.17 0)
+			(effects
+				(font
