File: pcb/main_MagicAlonso/CH340G_programmer.kicad_sch (KiCad schematic)
At the start: 15 parts, among them J13 USB_C_Receptacle_USB2.0_16P, J14 UART_Out, J15 USB_Out, J16 USB_B_Micro, U4 CH340C

Commit message: more pcb stuff ha
Parts:
- J15: footprint Connector_PinSocket_2.54mm:PinSocket_1x05_P2.54mm_Vertical -> MixLib:USB_Adapter_Board
Connections:
- net VMus is gone; now on net VMusB: J15.5 (Pin_5)
Changed lines of the file:
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@@
 		)
 	)
-	(label "VMus"
+	(label "VMusB"
 		(at 83.058 88.646 180)
 		(effects
@@
 			)
 		)
-		(property "Footprint" "Connector_PinSocket_2.54mm:PinSocket_1x05_P2.54mm_Vertical"
+		(property "Footprint" "MixLib:USB_Adapter_Board"
 			(at 89.408 93.726 0)
 			(effects

Commit message: pcb pcb
Parts:
- removed J15: USB_Out, MixLib:USB_Adapter_Board, symbol Connector:Conn_01x05_Pin
Connections:
- no-connect marks 11 -> 10
Other:
- moved on the sheet: J14

Commit message: pcb sync
Parts:
- C13: footprint Capacitor_SMD:C_0603_1608Metric_Pad1.08x0.95mm_HandSolder -> Capacitor_SMD:C_0805_2012Metric
- C14: footprint Capacitor_SMD:C_0805_2012Metric -> Capacitor_SMD:C_0603_1608Metric
Changed lines of the file:
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@@
 			)
 		)
-		(property "Footprint" "Capacitor_SMD:C_0805_2012Metric"
+		(property "Footprint" "Capacitor_SMD:C_0603_1608Metric"
 			(at 137.16 45.72 0)
 			(effects
@@
 			)
 		)
-		(property "Footprint" "Capacitor_SMD:C_0603_1608Metric_Pad1.08x0.95mm_HandSolder"
+		(property "Footprint" "Capacitor_SMD:C_0805_2012Metric"
 			(at 129.54 45.72 0)
 			(effects

Commit message: PCB components order
Parts:
- removed C15: 10uF, Capacitor_Tantalum_SMD:CP_EIA-3216-10_Kemet-I_HandSolder, symbol Device:C_Small
- removed C16: 100nF, Capacitor_SMD:C_0805_2012Metric, symbol Device:C_Small
- R10, R11, R12, R13: footprint Resistor_SMD:R_0805_2012Metric -> Resistor_SMD:R_0603_1608Metric
Other:
- moved on the sheet: D6

Commit message: pcb
Parts:
- J14: footprint Connector_JST:JST_XH_B4B-XH-A_1x04_P2.50mm_Vertical -> Connector_JST:JST_XH_S4B-XH-A_1x04_P2.50mm_Horizontal
Changed lines of the file:
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@@
 			)
 		)
-		(property "Footprint" "Connector_JST:JST_XH_B4B-XH-A_1x04_P2.50mm_Vertical"
+		(property "Footprint" "Connector_JST:JST_XH_S4B-XH-A_1x04_P2.50mm_Horizontal"
 			(at 92.71 86.36 0)
 			(effects
