File: pcb/main_MagicAlonso/main_MagicAlonso.kicad_sch (KiCad schematic)
At the start: 62 parts, among them J1 XT30PW-M, J10 ESC1, J11 ESC2, J12 ESC3, J17 aux0, J18 aux2, J19 aux1, J2 MPU6050, J3 OLED, J4 Encoder1, J5 Encoder2, J6 ESC1_VM, J7 ESC2_VM, J8 ESC3_VM, J9 Sensors, Q1 IRLML2502, SW1 Power_SW, SW2 EN_Push, SW3 Boot_SW, SW4 BUTTON_Push, U1 ESP32-WROOM-32E, U2 ACS712-30A, U3 ACS712-20A

Commit message: pcb changes
Connections:
- net VM: no longer R4.2
- net Vb: now also R4.2
Changed lines of the file:
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@@
 			"AAAAAAAAAAAAAAAAAAAAAAAAAAAAAAAAAAAAAAAAAAAAAAAAAAAAAAAAAAAAAAAAAAAAAAAAAAAA"
 			"AAAAAAAAAAAAAAAAAAAAAAAAAAAAAAAAAAAAAAAAAAAAAAAAAAAAAAAAAAAAAAAAAAAAAAAAAAAA"
-			"AAAAAA=="
+			"AAAAAJeRwsGEcSs+uCzrQJWRwsHz/C4+AAAAAAAAAAAAAAAAAAAAAAAAAAAROgIAAQAAAPh/AACQ"
+			"EumgfAsGgEUD60CXkcLBHaAqPtAh60CVkcLBiysuPiDsD8acAgAA4OgPxpwCAAAAAAAAAAAAAAAA"
+			"AAAAAAAAlBLtoAAMBoDmFutA8NHCwfH8Lj7ak+1AlZHCwfP8Lj4AAAAAAAAAAAAAAAAAAAAAAAAA"
+			"AA06AgACAAAA3aY9QZgS4aAEDQaA/gvrQPDRwsElty4+ixLrQJWRwsHz/C4+AAAAAAAAAAAAAAAA"
+			"AAAAAAAAAAAgOgIAAgAAAAAAAICcEuWgAg4GgOYW60CXkcLBUrcrPq157UCVkcLB8/wuPgAAAAAA"
+			"AAAAAAAAAAAAAAAAAAAADDoCAAEAAADepj1BgBL5oAUPBoBFA+tA8NHCwbzlLT4ADOtAlZHCwSe3"
+			"Lj5g5g/GnAIAAKDlD8acAgAAAgAAAAAAAAAAAAAAAAAAAIQS/aAAEAaAiRLrQJeRwsG3Kys+0CHr"
+			"QJWRwsHz/C4+AAAAAAAAAAAAAAAAAAAAAAAAAAATOgIAAQAAAAAAAICIEvGgABEGgKEH60Dw0cLB"
+			"iSsuPgAM60CVkcLBJ7cuPgAAAAAAAAAAAAAAAAAAAAAAAAAAIjoCAAIAAADjZG/BjBL1oGQSBoDO"
+			"IetAl5HCwbcrKz4tJutAubrBwYZxKz4AAAAAAAAAAAAAAAAAAAAAAAAAAP85AgACAAAA8NBRwbAS"
+			"yaAFEwaA6P7qQJeRwsGycSg+cx3rQJWRwsG7iCw+YOkPxpwCAABg7A/GnAIAAAIAAAAAAAAAAAAA"
+			"AAAAAIC0Es2g3RQGgEUD60Dw0cLBvOUtPqMH60CVkcLBiysuPgAAAAAAAAAAAAAAAAAAAAAAAAAA"
+			"JDoCAAIAAAAAAAAAuBLBoAAVBoAVGetAl5HCwRpDKT50HetAubrBwR+gKj6g8A/GnAIAAGDwD8ac"
+			"AgAAAgAAAAAAAAAAAAAAAAAAALwSxaAAFgaA5hbrQJeRwsFStys+FTHrQJWRwsHz/C4+AAAAAAAA"
+			"AAAAAAAAAAAAAAAAAAAQOgIAAQAAAPh/AACgEtmgnBcGgP4L60CXkcLBtysrPi0m60CVkcLB8/wu"
+			"PqDjD8acAgAAYOoPxpwCAAAAAAAAAAAAAAAAAADkAeI+pBLdoK8YBoBDG+tAl5HCwbXOKT5zHetA"
+			"ubrBwR+gKj4AAAAAAAAAAAAAAAAAAAAAAAAAAAQ6AgABAAAA/////6gS0aD/GQaAEzHrQJeRwsFS"
+			"tys+rXntQLm6wcFUtys+AAAAAAAAAAAAAAAAAAAAAAAAAAD5OQIAAgAAAPh/AACsEtWgZRoGgHId"
+			"60CXkQ=="
 		)
 	)
@@
 		)
 	)
+	(label "Vb"
+		(at 27.94 118.11 180)
+		(effects
+			(font
+				(size 1.27 1.27)
+			)
+			(justify right bottom)
+		)
+	)
 	(label "CurrESC1&2"
 		(at 302.26 38.1 0)
@@
 		)
 	)
-	(label "VM"
-		(at 27.94 118.11 180)
-		(effects
-			(font
-				(size 1.27 1.27)
-				(thickness 0.254)
-				(bold yes)
-			)
-			(justify right bottom)
-		)
-	)

Commit message: PCB components order
Parts:
- removed C25: 100nF, Capacitor_SMD:C_0805_2012Metric, symbol Device:C_Small
- removed D4: WS2812B, LED_SMD:LED_WS2812B_PLCC4_5.0x5.0mm_P3.2mm, symbol LED:WS2812B
- removed J6: ESC1_VM, TerminalBlock_Phoenix:TerminalBlock_Phoenix_PT-1,5-2-3.5-H_1x02_P3.50mm_Horizontal, symbol Connector:Screw_Terminal_01x02
- removed J7: ESC2_VM, TerminalBlock_Phoenix:TerminalBlock_Phoenix_PT-1,5-2-3.5-H_1x02_P3.50mm_Horizontal, symbol Connector:Screw_Terminal_01x02
- removed J8: ESC3_VM, TerminalBlock_Phoenix:TerminalBlock_Phoenix_PT-1,5-2-3.5-H_1x02_P3.50mm_Horizontal, symbol Connector:Screw_Terminal_01x02
- removed R6: 100, Resistor_SMD:R_0805_2012Metric, symbol Device:R_Small
- added J15: ESC_VM, TerminalBlock_Phoenix:TerminalBlock_Phoenix_PT-1,5-6-3.5-H_1x06_P3.50mm_Horizontal, symbol Connector:Screw_Terminal_01x06
- C5, C6: footprint Capacitor_SMD:C_0805_2012Metric -> Capacitor_SMD:C_0603_1608Metric
- J10, J11, J12: footprint Connector_JST:JST_XH_B2B-XH-A_1x02_P2.50mm_Vertical -> Connector_JST:JST_XH_S2B-XH-A_1x02_P2.50mm_Horizontal
- J17, J18, J19: footprint Connector_JST:JST_XH_B3B-XH-A_1x03_P2.50mm_Vertical -> MixLib:PinHeader_1x03_P2.54-SMD
- J3: footprint Connector_JST:JST_XH_B4B-XH-A_1x04_P2.50mm_Vertical -> Connector_PinSocket_2.54mm:PinSocket_1x04_P2.54mm_Vertical
Connections:
- net ESC1&2_VM: now also J15.1 (Pin_1), J15.2 (Pin_2)
- net ESC3_VM: now also J15.3 (Pin_3)
- net GND: now also J15.4 (Pin_4), J15.5 (Pin_5), J15.6 (Pin_6)
- net RX: now also U1.35 (TXD0/IO1); no longer U1.34 (RXD0/IO3)
- net TX: now also U1.34 (RXD0/IO3); no longer U1.35 (TXD0/IO1)
- net at D3.2 (DOUT): now also D5.4 (DIN)
Other:
- moved on the sheet: C24, C26, D3, D5, J10, J11, J12, R5, R7

Commit message: PCB advancements
Parts:
- added H10, H9: M2, MountingHole:MountingHole_2.2mm_M2, symbol Mechanical:MountingHole
- H7, H8: value M3 -> M2; footprint MountingHole:MountingHole_3mm -> MountingHole:MountingHole_2.2mm_M2
Connections:
- net CurrESC1&2: now also U1.5 (SENSOR_VN)
- net CurrESC2: now also U1.4 (SENSOR_VP)
- net ESC_1: now also U1.8 (IO32)
- net ESC_2: now also U1.9 (IO33)
- net ESC_3: now also U1.10 (IO25)
- net Enc1: now also U1.6 (IO34)
- net Enc2: now also U1.7 (IO35)
- net LEDs: now also U1.37 (IO23)
Other:
- note added: "X"
- moved on the sheet: H3, H4, H5, H6, H7, H8

Commit message: pcb
Parts:
- removed J3: OLED, Connector_PinSocket_2.54mm:PinSocket_1x04_P2.54mm_Vertical, symbol Connector:Conn_01x04_Pin
- J2: footprint Connector_PinSocket_2.54mm:PinSocket_1x04_P2.54mm_Vertical -> MixLib:MPU6050_Module
- R4: footprint Resistor_SMD:R_0805_2012Metric -> Resistor_SMD:R_1206_3216Metric
Connections:
- net CurrESC1&2: no longer U1.5 (SENSOR_VN)
- net CurrESC2: no longer U1.4 (SENSOR_VP)
- net ESC_1: no longer U1.8 (IO32)
- net ESC_2: no longer U1.9 (IO33)
- net ESC_3: no longer U1.10 (IO25)
- net Enc1: no longer U1.6 (IO34)
- net Enc2: no longer U1.7 (IO35)
- net LEDs: no longer U1.37 (IO23)
- net D_LED: now reaches D3.2 (DOUT), D5.4 (DIN)
Other:
- note removed: "X"
- moved on the sheet: C10, C24, C26, C6, D3, D5, J2, J4, J5, R5, R7, U3

Commit message: mais avances en la pcb
Parts:
- C8: footprint Capacitor_SMD:C_0805_2012Metric -> Capacitor_SMD:C_0603_1608Metric
Connections:
- net BUTTON: now also U1.4 (SENSOR_VP)
- net ESC_1: now also U1.14 (IO12)
- net ESC_2: now also U1.16 (IO13)
- net ESC_3: now also U1.23 (IO15)
- net Enc1: now also U1.26 (IO4)
- net Enc2: now also U1.27 (IO16)
Other:
- note added: "X"
Changed lines of the file:
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@@
 		)
 	)
+	(text "X"
+		(exclude_from_sim no)
+		(at 354.838 29.972 0)
+		(effects
+			(font
+				(size 1.27 1.27)
+				(thickness 0.254)
+				(bold yes)
+			)
+		)
+	)
 	(text "(IO12)"
 		(exclude_from_sim no)
@@
 		)
 	)
+	(text "X"
+		(exclude_from_sim no)
+		(at 311.912 27.178 0)
+		(effects
+			(font
+				(size 1.27 1.27)
+				(thickness 0.254)
+				(bold yes)
+			)
+		)
+	)
 	(text "Passive Buzzer"
 		(exclude_from_sim no)
@@
 		)
 	)
+	(text "X"
+		(exclude_from_sim no)
+		(at 309.118 43.688 0)
+		(effects
+			(font
+				(size 1.27 1.27)
+				(thickness 0.254)
+				(bold yes)
+			)
+		)
+	)
+	(text "X"
+		(exclude_from_sim no)
+		(at 309.118 46.482 0)
+		(effects
+			(font
+				(size 1.27 1.27)
+				(thickness 0.254)
+				(bold yes)
+			)
+		)
+	)
+	(text "X"
+		(exclude_from_sim no)
+		(at 354.838 32.512 0)
+		(effects
+			(font
+				(size 1.27 1.27)
+				(thickness 0.254)
+				(bold yes)
+			)
+		)
+	)
 	(text "Mounting\nHoles\n"
 		(exclude_from_sim no)
@@
 		)
 	)
+	(text "X"
+		(exclude_from_sim no)
+		(at 354.838 27.178 0)
+		(effects
+			(font
+				(size 1.27 1.27)
+				(thickness 0.254)
+				(bold yes)
+			)
+		)
+	)
 	(text "Boot "
 		(exclude_from_sim no)
@@
 	(wire
 		(pts
+			(xy 273.05 55.88) (xy 271.78 55.88)
+		)
+		(stroke
+			(width 0)
+			(type default)
+		)
+	)
+	(wire
+		(pts
 			(xy 86.36 31.75) (xy 86.36 33.02)
 		)
@@
 	(wire
 		(pts
+			(xy 273.05 48.26) (xy 271.78 48.26)
+		)
+		(stroke
+			(width 0)
+			(type default)
+		)
+	)
+	(wire
+		(pts
 			(xy 57.15 95.25) (xy 57.15 96.52)
 		)
@@
 	(wire
 		(pts
+			(xy 273.05 45.72) (xy 271.78 45.72)
+		)
+		(stroke
+			(width 0)
+			(type default)
+		)
+	)
+	(wire
+		(pts
+			(xy 273.05 53.34) (xy 271.78 53.34)
+		)
+		(stroke
+			(width 0)
+			(type default)
+		)
+	)
+	(wire
+		(pts
 			(xy 85.09 115.57) (xy 85.09 116.84)
 		)
@@
 	(wire
 		(pts
+			(xy 273.05 40.64) (xy 271.78 40.64)
+		)
+		(stroke
+			(width 0)
+			(type default)
+		)
+	)
+	(wire
+		(pts
 			(xy 80.01 167.64) (xy 80.01 166.37)
 		)
@@
 			"AHcFgA1kP0BEltfA6XcbPVxIQEAcJNfAYTMhPWDubNnkAgAAINhs2eQCAAACAAAAAAAAAAAAAAAA"
 			"AAAAleAFNAB4BYANZD9Aa4jXwF8zIT3NQ0BAsjfXwGEzIT0AAAAAAAAAAAAAAAAAAAAAAAAAAMyi"
-			"AQABAA=="
+			"AQABADcAegBqAEgAQwBwAHgARwBiAHUAeABoAFIAUgBnAC8ALwA3ADkAZQBYAHEAbQBNAFUARgB2"
+			"AE0AZgByAGsANQBzAGIAYQA2AEUARwBzAFIAMAB3ADEAbgBqAEsASAA0AG8AegArAEMANQByAG4A"
+			"MwByAGoAOQB1AEQAYwB3AEcAVQAwAG4AZgBuAEQANwBIAEUATgA4AFkAVgBjAFUASQBQAGEATwBM"
+			"ACsASQBWADgATQBDAG8AOQAyAFEAOABpAC8AdQBaAFgAZQAwAEoAOAAyADIAeAA4AEsAawBYAHIA"
+			"dgBFAGwAdAByAFQAdwA1AFYAawBPAG8AQwByAHgAVABOAHoARABCAGEAMQB6AHYAOQB2AG0AeAB2"
+			"AFoARABCAEEAQQBPAHgAcwBuACsAbQA1AHQAdABBAE0AZABtAHgAVQArAFAAUgBBAEgAMABYACsA"
+			"NgBjAHkANgArAC8AZgBJAGwAcgBVAHYAVwBMAEEAWABxAEwAWQBtAHMAcgB2ACsAVgBnAFoASwBu"
+			"ADUAbQBsAFYAegB6AC8AdQBlADIAQgBYADAAdwBGAFQAMQBUAEIARABxAEMAUQA5AFkAegBGAHIA"
+			"eAB5AEoARQBqAEsAWABaAEsAQwBEAFIAVwBOAHUAVwBEADAAZAAzAGUAcwBxAG8AOQBBADYAQQA1"
+			"AGIAZgAzAHUAbABtAFYAdABhAFgAZABaAFcAMwBaAHAAMAA1AHoAYgAwADAAQwBoADgAdABEAHgA"
+			"aQBhAE8ARABJADEATABwAEoAZgBtAFcASABTAHUANwBMAGwAMwBaAGwAawBTAFcAZAAvAGUATwBE"
+			"AEIAZABtAEMATQBoADEARgA2ACsAOQA1ADkARAB3AHcAWQBIAGgAbAB1AGEAbQBTADkAWgAwAEoA"
+			"MAA1AEEARQArAFgAZwBsADAAZQBHAHgANABxAFYAdwBuAFMAeAB2AGIAVgA1ADkAWgBLADIANQA2"
+			"ADkAcQBiADAAbABiAEEARgBwAGoAbwBlAHYARQBkAEYARQBxAGIAUwBaADQAagAwADUAVwB4AGcA"
+			"bwB6AEEAQwA1AGUAMQBRAEYAZwBZAGoAWQA2ADcAagBhAGoAeQArAEoANgBtAHUAMgBaAHQAbQBQ"
+			"AGoAMwBjAGIAYwBmAGIAcgBxAEwANABwAFEAeQA0AEYAYQBTAEoAWgBOAE4ATAArADgAYgBmAEgA"
+			"YgBrAGQARAA2AHEAegAvAHQAQgAzAEQAUgBoAHMANQBMAE4ANwBTAHMAWABwAEkAZABHAHAAcwBH"
+			"ADAARAB0AGMAUwBSAEQAcQA0AGUARgBLAGoARgBEAG4AZgB0AFMAaQBaAEgATgBQADAANABuAFIA"
+			"YQBRAAAAAAAAAAAAAAAAAAAAAAAAAAAAAAAAAAAAAAAAAAAAAAAAAAAAAAAAAAAAAAAAAAAAAAAA"
+			"AAAAAAAAAAAAAAAAAAAAAAAAAAAAAAAAAAAAAAAAAAAAAAAAAAAAAAAAAAAAAAAAAAAAAAAAAAAA"
+			"AAAAAAAAAAAAAAAAAAAAAAAAAAAAAAAAAAAAAAAAAAAAAAAAAAAAAAAAAAAAAAAAAAAAAAAAAAAA"
+			"AAAAAAAAAAAAAAAAAAAAAAAAAAAAAAAAAAAAAAAAAAAAAAAAAAAAAAAAAAAAAAAAAAAAAAAAAAAA"
+			"AAAAAAAAAAAAAAAAAAAAAAAAAAAAAAAAAAAAAAAAAAAAAAAAAAAAAAAAAAAAAAAAAAAAAAAAAAAA"
+			"AAAAAAAAAAAAAAAAAAAAAAAAAAAAAAAAAAAAAAAAAAAAAAAAAAAAAAAAAAAAAAAAAAAAAAAAAAAA"
+			"AAAAAAAAAAAAAAAAAAAAAAAAAAAAAAAAAAAAAAAAAAAAAAAAAAAAAAAAAAAAAAAAAAAAAAAAAAAA"
+			"AAAAAAAAAAAAAAAAAAAAAAAAAAAAAAAAAAAAAAAAAAAAAAAAAAAAAAAAAAAAAAAAAAAAAAAAAAAA"
+			"AAAAAAAAAAAAAAAAAAAAAAAAAAAAAAAAAAAAAAAAAAAAAAAAAAAAAAAAAAAAAAAAAAAAAAAAAAAA"
+			"AAAAAAAAAAAAAAAAAAAAAAAAAAAAAAAAAAAAAAAAAAAAAAAAAAAAAAAAAAAAAAAAAAAAAAAAAAAA"
+			"AAAAAAAAAAAAAAAAAAAAAAAAAAAAAAAAAAAAAAAAAAAAAAAAAAAAAAAAAAAAAAAAAAAAAAAAAAAA"
+			"AAAAAAAAAAAAAAAAAAAAAAAAAAAAAAAAAAAAAAAAAAAAAAAAAAAAAAAAAAAAAAAAAAAAAAAAAAAA"
+			"AAAAAAAAAAAAAAAAAAAAAAAAAAAAAAAAAAAAAAAAAAAAAAAAAAAAAAAAAAAAAAAAAAAAAAAAAAAA"
+			"AAAAAAAAAAAAAAAAAAAAAAAAAAAAAAAAAAAAAAAAAAAAAAAAAAAAAAAAAAAAAAAAAAAAAAAAAAAA"
+			"AAAAAAAAAAAAAAAAAAAAAAAAAAAAAAAAAAAAAAAAAAAAAAAAAAAAAAAAAAAAAAAAAAAAAAAAAAAA"
+			"AAAAAAAAAAAAAAAAAAAAAAAAAAAAAAAAAAAAAAAAAAAAAAAAAAAAAAAAAAAAAAAAAAAAAAAAAAAA"
+			"AAAAAAAAAAAAAAAAAAAAAAAAAAAAAAAAAAAAAAAAAAAAAAAAAAAAAAAAAAAAAAAAAAAAAAAAAAAA"
+			"AAAAAAAAAAAAAAAAAAAAAAAAAAAAAAAAAAAAAAAAAAAAAAAAAAAAAAAAAAAAAAAAAAAAAAAAAAAA"
+			"AAAAAA=="
 		)
 	)
@@
 	)
 	(label "Enc1"
-		(at 302.26 41.91 0)
+		(at 273.05 40.64 0)
 		(effects
 			(font
@@
 		)
 	)
+	(label "ESC_2"
+		(at 273.05 48.26 0)
+		(effects
+			(font
+				(size 1.27 1.27)
+			)
+			(justify left bottom)
+		)
+	)
 	(label "Data_S3"
 		(at 323.85 31.75 0)
@@
 		)
 	)
+	(label "ESC_1"
+		(at 273.05 45.72 0)
+		(effects
+			(font
+				(size 1.27 1.27)
+			)
+			(justify left bottom)
+		)
+	)
 	(label "ESC1&2_VM"
 		(at 125.73 161.29 180)
@@
 		)
 	)
+	(label "Enc1"
+		(at 302.26 46.99 0)
+		(effects
+			(font
+				(size 1.27 1.27)
+			)
+			(justify left bottom)
+		)
+	)
 	(label "SCL"
 		(at 161.29 82.55 0)
@@
 		)
 	)
+	(label "Enc2"
+		(at 273.05 55.88 0)
+		(effects
+			(font
+				(size 1.27 1.27)
+			)
+			(justify left bottom)
+		)
+	)
+	(label "BUTTON"
+		(at 240.03 41.91 180)
+		(effects
+			(font
+				(size 1.27 1.27)
+			)
+			(justify right bottom)
+		)
+	)
 	(label "CurrESC1&2"
 		(at 57.15 86.36 0)
@@
 		)
 	)
+	(label "ESC_3"
+		(at 273.05 53.34 0)
+		(effects
+			(font
+				(size 1.27 1.27)
+			)
+			(justify left bottom)
+		)
+	)
 	(label "Data_S3"
 		(at 25.4 168.91 0)
@@
 			)
 		)
-		(property "Footprint" "Capacitor_SMD:C_0805_2012Metric"
+		(property "Footprint" "Capacitor_SMD:C_0603_1608Metric"
 			(at 231.14 73.66 0)
 			(effects

Commit message: update PCB
Connections:
- net CurrESC1&2: now also U1.13 (IO14)
- net CurrESC2: now also U1.12 (IO27)
- net Data_0aux: now also U1.37 (IO23)
- net Data_1aux: now also U1.31 (IO19)
- net Data_2aux: now also U1.30 (IO18)
Other:
- moved on the sheet: U1

Commit message: Update PCB
Connections:
- net BUZ: now also U1.26 (IO4)
- net Data_1aux: no longer U1.31 (IO19)
- net Data_2aux: no longer U1.30 (IO18)
- net Data_S0: now also U1.31 (IO19)
- net Data_S1: now also U1.30 (IO18)
- net Data_S2: now also U1.28 (IO17)
- net Data_S3: now also U1.27 (IO16)
- net Enc1: now also U1.6 (IO34); no longer U1.26 (IO4)
- net Enc2: now also U1.5 (SENSOR_VN); no longer U1.27 (IO16)
Changed lines of the file:
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@@
 		)
 	)
-	(text "X"
-		(exclude_from_sim no)
-		(at 357.886 41.148 0)
-		(effects
-			(font
-				(size 1.27 1.27)
-				(thickness 0.254)
-				(bold yes)
-			)
-		)
-	)
 	(text "Strapping Pin\n\nGPIO0\nGPIO2\nMTDI\nMTDO\nGPIO5"
 		(exclude_from_sim no)
@@
 	(text "X"
 		(exclude_from_sim no)
-		(at 357.886 35.814 0)
-		(effects
-			(font
-				(size 1.27 1.27)
-				(thickness 0.254)
-				(bold yes)
-			)
-		)
-	)
-	(text "X"
-		(exclude_from_sim no)
 		(at 354.838 29.972 0)
 		(effects
@@
 	(text "X"
 		(exclude_from_sim no)
+		(at 334.772 41.148 0)
+		(effects
+			(font
+				(size 1.27 1.27)
+				(thickness 0.254)
+				(bold yes)
+			)
+		)
+	)
+	(text "X"
+		(exclude_from_sim no)
 		(at 311.912 27.178 0)
 		(effects
@@
 		)
 	)
+	(text "X"
+		(exclude_from_sim no)
+		(at 330.708 27.178 0)
+		(effects
+			(font
+				(size 1.27 1.27)
+				(thickness 0.254)
+				(bold yes)
+			)
+		)
+	)
 	(text "I2C Connectíons"
 		(exclude_from_sim no)
@@
 		)
 	)
+	(text "X"
+		(exclude_from_sim no)
+		(at 334.772 35.814 0)
+		(effects
+			(font
+				(size 1.27 1.27)
+				(thickness 0.254)
+				(bold yes)
+			)
+		)
+	)
 	(text "Mounting\nHoles\n"
 		(exclude_from_sim no)
@@
 		)
 	)
+	(text "X"
+		(exclude_from_sim no)
+		(at 334.772 38.608 0)
+		(effects
+			(font
+				(size 1.27 1.27)
+				(thickness 0.254)
+				(bold yes)
+			)
+		)
+	)
 	(text "Battery Supply - 2S LiPo"
 		(exclude_from_sim no)
@@
 		)
 	)
+	(text "X"
+		(exclude_from_sim no)
+		(at 316.484 36.068 0)
+		(effects
+			(font
+				(size 1.27 1.27)
+				(thickness 0.254)
+				(bold yes)
+			)
+		)
+	)
 	(text "MCU"
 		(exclude_from_sim no)
@@
 		)
 	)
-	(text "Button"
+	(text "X"
 		(exclude_from_sim no)
-		(at 54.864 108.966 0)
+		(at 316.484 38.862 0)
 		(effects
 			(font
-				(size 2 2)
-				(thickness 0.25)
-				(italic yes)
+				(size 1.27 1.27)
+				(thickness 0.254)
+				(bold yes)
 			)
 		)
 	)
-	(text "X"
+	(text "Button"
 		(exclude_from_sim no)
-		(at 357.886 38.608 0)
+		(at 54.864 108.966 0)
 		(effects
 			(font
-				(size 1.27 1.27)
-				(thickness 0.254)
-				(bold yes)
+				(size 2 2)
+				(thickness 0.25)
+				(italic yes)
 			)
 		)
@@
 		)
 	)
+	(text "X"
+		(exclude_from_sim no)
+		(at 334.772 33.274 0)
+		(effects
+			(font
+				(size 1.27 1.27)
+				(thickness 0.254)
+				(bold yes)
+			)
+		)
+	)
 	(text "Bidirectionals"
 		(exclude_from_sim no)
@@
 	(wire
 		(pts
+			(xy 271.78 58.42) (xy 270.51 58.42)
+		)
+		(stroke
+			(width 0)
+			(type default)
+		)
+	)
+	(wire
+		(pts
 			(xy 223.52 30.48) (xy 223.52 31.75)
 		)
@@
 			"MgBhAFcATwA1ACsAdwBBAHQAZQBBAHYAeABhAGwAdwAwADEAQgBYADQAYwBlAE8AQwB1AGUAeAAz"
 			"AFEAQgA3ADQASwB1AEIAcgBZAEQANwB3AEwAKwBQAFkANQB6ADQARwA1AFcAcwBOAGEAVwBaAGUA"
-			"bgBkAA=="
+			"bgBkAAAAAAAAAAAAAAAAAAAAAAAAAAAAAAAAAAAAAAAAAAAAAAAAAAAAAAAAAAAAAAAAAAAAAAAA"
+			"AAAAAAAAAAAAAAAAAAAAAAAAAAAAAAAAAAAAAAAAAAAAAAAAAAAAAAAAAAAAAAAAAAAAAAAAAAAA"
+			"AAAAAAAAAAAAAAAAAAAAAAAAAAAAAAAAAAAAAAAAAAAAAAAAAAAAAAAAAAAAAAAAAAAAAAAAAAAA"
+			"AAAAAAAAAAAAAAAAAAAAAAAAAAAAAAAAAAAAAAAAAAAAAAAAAAAAAAAAAAAAAAAAAAAAAAAAAAAA"
+			"AAAAAAAAAAAAAAAAAAAAAAAAAAAAAAAAAAAAAAAAAAAAAAAAAAAAAAAAAAAAAAAAAAAAAAAAAAAA"
+			"AAAAAAAAAAAAAAAAAAAAAAAAAAAAAAAAAAAAAAAAAAAAAAAAAAAAAAAAAAAAAAAAAAAAAAAAAAAA"
+			"AAAAAAAAAAAAAAAAAAAAAAAAAAAAAAAAAAAAAAAAAAAAAAAAAAAAAAAAAAAAAAAAAAAAAAAAAAAA"
+			"AAAAAAAAAAAAAAAAAAAAAAAAAAAAAAAAAAAAAAAAAAAAAAAAAAAAAAAAAAAAAAAAAAAAAAAAAAAA"
+			"AAAAAAAAAAAAAAAAAAAAAAAAAAAAAAAAAAAAAAAAAAAAAAAAAAAAAAAAAAAAAAAAAAAAAAAAAAAA"
+			"AAAAAAAAAAAAAAAAAAAAAAAAAAAAAAAAAAAAAAAAAAAAAAAAAAAAAAAAAAAAAAAAAAAAAAAAAAAA"
+			"AAAAAAAAAAAAAAAAAAAAAAAAAAAAAAAAAAAAAAAAAAAAAAAAAAAAAAAAAAAAAAAAAAAAAAAAAAAA"
+			"AAAAAAAAAAAAAAAAAAAAAAAAAAAAAAAAAAAAAAAAAAAAAAAAAAAAAAAAAAAAAAAAAAAAAAAAAAAA"
+			"AAAAAAAAAAAAAAAAAAAAAAAAAAAAAAAAAAAAAAAAAAAAAAAAAAAAAAAAAAAAAAAAAAAAAAAAAAAA"
+			"AAAAAAAAAAAAAAAAAAAAAAAAAAAAAAAAAAAAAAAAAAAAAAAAAAAAAAAAAAAAAAAAAAAAAAAAAAAA"
+			"AAAAAAAAAAAAAAAAAAAAAAAAAAAAAAAAAAAAAAAAAAAAAAAAAAAAAAAAAAAAAAAAAAAAAAAAAAAA"
+			"AAAAAAAAAAAAAAAAAAAAAAAAAAAAAAAAAAAAAAAAAAAAAAAAAAAAAAAAAAAAAAAAAAAAAAAAAAAA"
+			"AAAAAAAAAAAAAAAAAAAAAAAAAAAAAAAAAAAAAAAAAAAAAAAAAAAAAAAAAAAAAAAAAAAAAAAAAAAA"
+			"AAAAAAAAAAAAAAAAAAAAAAAAAAAAAAAAAAAAAAAAAAAAAAAAAAAAAAAAAAAAAAAAAAAAAAAAAAAA"
+			"AAAAAGMAVgBYAEEAYwBIAHcANQBhAEoAYQBEAEsAWgBIAEQAMQA2AHAASwBtAHEAbwB0AGMAagBO"
+			"AG0AMABhAHYAWgBLAHoAegB1AFkAMgBoAEcAYgBUAGIAbQA1AE4AeABpAEkAeAA5AFUARgA3AEYA"
+			"UwBWAHgAeABoAEoAUgBpADAAYQBpAGUAQgBXAGIAYgBFAGkAagBSAEEAawArAFIAQwBKAHkAMQBo"
+			"AHAAagB3AEIAdwBsAHAAZwA3AHUAbQBjAFIAUABWAEYATABXAFUASQBLAG8ATQBRAFEAbwBpAEoA"
+			"TgB6AHEAUwBhAEYANgBlAHcAagAwAEsAeQBZAE4AUgBrAGYAbwBoAFgARQB0AFoAMwBJAEMAaQBL"
+			"AHUAbQB4AEMAaABJAFAAQQBNAG8AagBGAGIAYQAwAG0AVgBBAEkARQAyAGoAVABmAEcAWgBGAG0A"
+			"VwBEAEIAOQBUAHQAMwA3AEsATgB5AGUAdwBFAHQAZwBhAFkAdwB5AEkAbQBMAGkAZgBGADEAdABi"
+			"AFcAMABFAFQAUwBEAFYAWgA1AGcAQgBzAGIARwA1AFcAVgBiAFYAcgB6ADIANABmAGcAcwBTAFEA"
+			"NwBDAHcAVgBtAGwAQwBPAGkAdgBpAG0AcwBjAFoAcQBXAHMAYwBXAFoALwBpAFUAdgA1AFIASQBh"
+			"AHgASwB4ADEAbgBVAGQAUQBsAGcAYQBEAFAAYgB1ADMAWAB2ADgAMgBEAEUAVgBTAGEASAB0AFIA"
+			"TwBTAHkATABIAE8AWgBNAFoAYQBVAHEAcQBvAFUASQBFAFEAZgBHAGgARwBGAFMAaABTAEoAeABs"
+			"AHAAcgBqAEEASgBCAHgASAB0AHYAagBlADIAUwB2AGoAVABQAHMAdQBGAGcAcwBMAFcAMQBSAGMA"
+			"eABGAFUAVABqAG4AbQBKAG4ANgBTADIAMQBqAGYAbABJAEYAaQBwAEkAbwBvADYAWABQAC8AWAA0"
+			"AC8AUABSAFAANwBFAEsASQBJAGkASgBnAG8AeABsAGgAWABsAFkAbwBrADQAVwAxAFoAbABpAG0A"
+			"bgBQAG8AbwBrAGUASgBlAGcAYgBWAG4AVgBqAGYAZABKADMAaABoAGoAZwBFAHEAZQBaAFYARwBr"
+			"AGIAcAByAEUATgBBADIAMwBBAHMATQBaAFoAeQB6AHkASQByAEYAYQBFAEcAQwBRAFoAWgBsAHoA"
+			"MgBkAHEASgBFADkARgA3AHcANgBiAEkAYwAyAEsAYQBUAEMAYQBUAHkAVgBhAGUAdQBiADcAcgBz"
+			"ADIARwBKAE0AaABnAE0AMABvAEcAUgB5AEoAcgAzAHYAaQB6AEwASwBOAEcAdwBtAGIAWAB3AHAA"
+			"egAxAA=="
 		)
 	)
@@
 		)
 	)
-	(label "Enc1"
-		(at 271.78 40.64 0)
-		(effects
-			(font
-				(size 1.27 1.27)
-			)
-			(justify left bottom)
-		)
-	)
 	(label "Data_0aux"
 		(at 77.47 163.83 0)
@@
 	)
 	(label "Data_S0"
-		(at 323.85 39.37 0)
+		(at 323.85 41.91 0)
 		(effects
 			(font
@@
 	)
 	(label "Data_S1"
-		(at 323.85 36.83 0)
+		(at 323.85 39.37 0)
 		(effects
 			(font
@@
 		)
 	)
+	(label "Data_S1"
+		(at 271.78 60.96 0)
+		(effects
+			(font
+				(size 1.27 1.27)
+			)
+			(justify left bottom)
+		)
+	)
 	(label "ESC_2"
 		(at 271.78 48.26 0)
@@
 	)
 	(label "Data_S3"
-		(at 323.85 31.75 0)
+		(at 271.78 55.88 0)
 		(effects
 			(font
@@
 	)
 	(label "Data_S2"
-		(at 323.85 34.29 0)
+		(at 323.85 36.83 0)
 		(effects
 			(font
@@
 	)
 	(label "CurrESC2"
-		(at 302.26 35.56 0)
+		(at 302.26 36.83 0)
 		(effects
 			(font
@@
 		)
 	)
+	(label "Enc1"
+		(at 271.78 86.36 0)
+		(effects
+			(font
+				(size 1.27 1.27)
+			)
+			(justify left bottom)
+		)
+	)
 	(label "CurrESC1&2"
 		(at 271.78 50.8 0)
@@
 		)
 	)
+	(label "CurrESC1&2"
+		(at 302.26 39.37 0)
+		(effects
+			(font
+				(size 1.27 1.27)
+			)
+			(justify left bottom)
+		)
+	)
 	(label "Data_SIG"
 		(at 25.4 166.37 0)
@@
 		)
 	)
+	(label "BUZ"
+		(at 271.78 40.64 0)
+		(effects
+			(font
+				(size 1.27 1.27)
+			)
+			(justify left bottom)
+		)
+	)
+	(label "Data_S0"
+		(at 271.78 63.5 0)
+		(effects
+			(font
+				(size 1.27 1.27)
+			)
+			(justify left bottom)
+		)
+	)
 	(label "SCL"
 		(at 161.29 82.55 0)
@@
 		)
 	)
-	(label "BUZ"
-		(at 323.85 27.94 0)
+	(label "Data_S2"
+		(at 271.78 58.42 0)
 		(effects
 			(font
@@
 		)
 	)
-	(label "Data_1aux"
-		(at 25.4 163.83 0)
+	(label "BUZ"
+		(at 323.85 27.94 0)
 		(effects
 			(font
@@
 		)
 	)
-	(label "Data_2aux"
-		(at 271.78 60.96 0)
+	(label "Data_1aux"
+		(at 25.4 163.83 0)
 		(effects
 			(font
@@
 	)
 	(label "Enc2"
-		(at 271.78 55.88 0)
+		(at 238.76 44.45 180)
 		(effects
 			(font
 				(size 1.27 1.27)
 			)
-			(justify left bottom)
+			(justify right bottom)
 		)
 	)
@@
 		)
 	)
-	(label "Data_1aux"
-		(at 271.78 63.5 0)
+	(label "RX"
+		(at 271.78 33.02 0)
 		(effects
 			(font
@@
 		)
 	)
-	(label "RX"
-		(at 271.78 33.02 0)
+	(label "Data_S3"
+		(at 323.85 34.29 0)
 		(effects
 			(font

Commit message: first PCB layout done
Parts:
- removed J17: aux0, MixLib:PinHeader_1x03_P2.54-SMD, symbol Connector:Conn_01x03_Pin
- removed J18: aux2, MixLib:PinHeader_1x03_P2.54-SMD, symbol Connector:Conn_01x03_Pin
- removed J19: aux1, MixLib:PinHeader_1x03_P2.54-SMD, symbol Connector:Conn_01x03_Pin
- added R6: 10k, Resistor_SMD:R_0805_2012Metric, symbol Device:R_Small
Connections:
- net BUZ: now also U1.9 (IO33); no longer U1.26 (IO4)
- net Data_1aux: now also U1.7 (IO35)
- net Data_2aux: now also U1.8 (IO32)
- net Data_SIG: now also U1.5 (SENSOR_VN)
- net Enc1: now also U1.11 (IO26); no longer U1.6 (IO34)
- net Enc2: now also U1.10 (IO25); no longer U1.5 (SENSOR_VN)
- net GND: now also R6.1
- net Data_0aux renamed Data_EN
- net Data_EN: now also R6.2
- no-connect marks 3 -> 6
