File: pcb/main_MagicAlonso/StepDown_2315.kicad_sch (KiCad schematic)
At the start: 18 parts, among them U6 Mini360

Commit message: PCB advancements
Parts:
- C22: value 22uF -> 10uF
Connections:
- net VCC_MP renamed VCC_SW
Other:
- moved on the sheet: C22
Changed lines of the file:
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@@
 	)
 	(junction
-		(at 110.49 39.37)
+		(at 109.22 39.37)
 		(diameter 0)
 		(color 0 0 0 0)
@@
 	(wire
 		(pts
+			(xy 109.22 39.37) (xy 118.11 39.37)
+		)
+		(stroke
+			(width 0)
+			(type default)
+		)
+	)
+	(wire
+		(pts
 			(xy 102.87 46.99) (xy 102.87 52.07)
 		)
@@
 	(wire
 		(pts
-			(xy 110.49 46.99) (xy 110.49 45.72)
+			(xy 109.22 46.99) (xy 109.22 45.72)
 		)
 		(stroke
@@
 	(wire
 		(pts
-			(xy 110.49 39.37) (xy 118.11 39.37)
-		)
-		(stroke
-			(width 0)
-			(type default)
-		)
-	)
-	(wire
-		(pts
 			(xy 82.55 55.88) (xy 82.55 57.15)
 		)
@@
 	(wire
 		(pts
-			(xy 102.87 39.37) (xy 110.49 39.37)
+			(xy 102.87 39.37) (xy 109.22 39.37)
 		)
 		(stroke
@@
 	(wire
 		(pts
-			(xy 110.49 39.37) (xy 110.49 40.64)
+			(xy 109.22 39.37) (xy 109.22 40.64)
 		)
 		(stroke
@@
 	(wire
 		(pts
-			(xy 102.87 46.99) (xy 110.49 46.99)
+			(xy 102.87 46.99) (xy 109.22 46.99)
 		)
 		(stroke
@@
 		)
 	)
-	(label "VCC_MP"
+	(label "VCC_SW"
 		(at 36.83 41.91 0)
 		(effects
@@
 	(symbol
 		(lib_id "Device:C_Small")
-		(at 110.49 43.18 0)
+		(at 109.22 43.18 0)
 		(unit 1)
 		(exclude_from_sim no)
@@
 		(dnp no)
 		(property "Reference" "C22"
-			(at 108.712 35.306 0)
+			(at 107.442 35.306 0)
 			(effects
 				(font
@@
 			)
 		)
-		(property "Value" "22uF"
-			(at 108.712 37.846 0)
+		(property "Value" "10uF"
+			(at 107.442 37.846 0)
 			(effects
 				(font
@@
 		)
 		(property "Footprint" "Capacitor_SMD:C_0805_2012Metric"
-			(at 110.49 43.18 0)
+			(at 109.22 43.18 0)
 			(effects
 				(font
@@
 		)
 		(property "Datasheet" "~"
-			(at 110.49 43.18 0)
+			(at 109.22 43.18 0)
 			(effects
 				(font
@@
 		)
 		(property "Description" "Unpolarized capacitor, small symbol"
-			(at 110.49 43.18 0)
-			(effects
-				(font
+			(at 109.22 43.18 0)
+			(effects
+				(font
