File: pcb/main_MagicAlonso/main_MagicAlonso.kicad_pcb (KiCad board)
At the start: 2 copper layers, 75.3 x 22 mm, 95 parts, among them J1 XT30PW-M, J10 ESC1, J11 ESC2, J12 ESC3, J13 USB_C_Receptacle_USB2.0_16P, J14 UART_Out, J15 USB_Out, J16 USB_B_Micro, J17 aux0, J18 aux2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

Commit message: yes, pcb
Parts:
- moved R1 245.6 mm to (267.8, 125.6), turned to 180 degrees
- moved H7 210.9 mm to (80.1, 243.3)
- moved H8 210.9 mm to (80.1, 250.8)
- moved D2 108.3 mm to (268.0, 128.1), turned to 180 degrees
- moved D1 78.5 mm to (238.6, 143.8), turned to 180 degrees
- moved R17 45.4 mm to (262.4, 130.6), turned to 180 degrees
- moved Rp1 44.5 mm to (261.4, 133.2), turned to -90 degrees
- moved C22 43.5 mm to (266.1, 140.3), turned to -90 degrees
- moved Rp2 43.3 mm to (259.5, 133.2), turned to -90 degrees
- moved R14 38.2 mm to (255.8, 132.1), turned to 180 degrees
- moved R15 35.5 mm to (253.2, 131.3), turned to 90 degrees
- moved R16 33.0 mm to (250.7, 135.5), turned to 90 degrees
- moved Rt1 22.2 mm to (251.5, 131.5), turned to 90 degrees
- moved C20 20.4 mm to (263.3, 133.3), turned to 90 degrees
- moved C19 20.3 mm to (256.8, 134.0)
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Connections:
- RV1 pad 1: unconnected-(RV1-Pad1) -> /StepDown_2315/Rt

Commit message: more pcb stuff ha
Parts:
- removed C1: 330uF, Capacitor_THT:CP_Radial_D8.0mm_P3.80mm
- added C28: 100uF, Capacitor_SMD:CP_Elec_6.3x5.4, F.Cu at (122.2, 233.0)
- C18, C19, C23: footprint Capacitor_SMD:C_0805_2012Metric -> Capacitor_SMD:C_0603_1608Metric
- C22: value 47uF -> 22uF; footprint Capacitor_SMD:CP_Elec_6.3x5.4 -> Capacitor_SMD:C_0805_2012Metric
- J1: footprint MixLib:XT30PW-M -> Connector_AMASS:AMASS_XT30U-M_1x02_P5.0mm_Vertical
- J15: footprint Connector_PinSocket_2.54mm:PinSocket_1x05_P2.54mm_Vertical -> MixLib:USB_Adapter_Board
- J6, J7, J8: footprint TerminalBlock_4Ucon:TerminalBlock_4Ucon_1x02_P3.50mm_Horizontal -> TerminalBlock_Phoenix:TerminalBlock_Phoenix_PT-1,5-2-3.5-H_1x02_P3.50mm_Horizontal
- R15, R16: footprint Resistor_SMD:R_0805_2012Metric -> Resistor_SMD:R_0603_1608Metric
- moved U6 224.6 mm to (71.8, 232.1), turned to 180 degrees
- moved R17 218.8 mm to (66.5, 228.1), turned to -90 degrees
- moved R15 214.0 mm to (64.3, 232.1), turned to 180 degrees
- moved C19 210.8 mm to (70.6, 232.8), turned to -90 degrees
- moved R16 210.7 mm to (64.4, 233.7), turned to 180 degrees
- moved Rt1 210.3 mm to (66.0, 230.5), turned to 180 degrees
- moved R14 210.0 mm to (70.2, 230.3)
- moved C18 209.8 mm to (66.2, 236.0)
- moved ST1 209.8 mm to (68.1, 233.4)
- moved Rp1 209.8 mm to (74.9, 229.3)
- moved Rp2 209.8 mm to (73.0, 229.3)
- moved L1 207.2 mm to (75.1, 234.6)
- moved C17 206.0 mm to (70.0, 236.9), turned to 0 degrees
- moved C23 201.6 mm to (69.4, 227.5), turned to 0 degrees
- moved RV1 190.9 mm to (79.3, 228.4)
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Connections:
- J15 pad 5: /CH340C/VMus -> /CH340C/VMusB
- RV1 pad 1: /StepDown_2315/Rt -> unconnected-(RV1-Pad1)
- U6 pad 1: /Vb -> (no net)
Routing:
- net /StepDown_2315/Rt: track 0.00 -> 0.71 mm
Other:
- board size 75.3 x 22 mm -> 117.5 x 122 mm
- board text added: "puedo mover conector mas adelante"

Commit message: pcb pcb
Parts:
- removed J15: USB_Out, MixLib:USB_Adapter_Board
- added REF**: R_1206_3216Metric, Resistor_SMD:R_1206_3216Metric, F.Cu at (157.1, 167.5)
- moved D6 85.2 mm to (135.7, 232.1), turned to -90 degrees
- moved D2 63.4 mm to (56.9, 168.8), turned to 0 degrees
- moved R1 61.8 mm to (56.9, 170.8), turned to 0 degrees
- moved R11 59.8 mm to (145.0, 155.1)
- moved R10 51.3 mm to (154.6, 153.1)
- moved R12 49.6 mm to (159.5, 155.6)
- moved R13 48.2 mm to (160.8, 159.1)
- moved U4 46.8 mm to (148.3, 165.7), turned to 180 degrees
- moved J14 43.0 mm to (133.0, 170.1)
- moved C14 18.2 mm to (181.5, 150.1)
- moved C15 18.2 mm to (189.3, 156.8)
- moved C16 18.2 mm to (181.5, 153.1)
- moved D7 18.2 mm to (175.2, 155.4)
- moved H8 11.8 mm to (102.0, 244.6), turned to 180 degrees
- moved F1 6.95 mm to (49.9, 169.8), turned to 90 degrees
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Connections:
- J6 pad 1: /ESC1&2_VM -> GND
- J6 pad 2: GND -> /ESC1&2_VM
- J7 pad 1: /ESC1&2_VM -> GND
- J7 pad 2: GND -> /ESC1&2_VM
- J8 pad 1: /ESC3_VM -> GND
- J8 pad 2: GND -> /ESC3_VM
- U6 pad 1: (no net) -> /Vb
Routing:
- net /CH340C/D-: track 0.00 -> 88.3 mm
- net /CH340C/D+: track 0.00 -> 83.5 mm
- net /CH340C/VMusC: track 0.00 -> 16.7 mm
- net /StepDown_2315/Rt: track 0.71 -> 0.00 mm

Commit message: pcb sync
Parts:
- C10, C5, C6, C9: moved to B.Cu
- C13: footprint Capacitor_SMD:C_0603_1608Metric_Pad1.08x0.95mm_HandSolder -> Capacitor_SMD:C_0805_2012Metric
- C14: footprint Capacitor_SMD:C_0805_2012Metric -> Capacitor_SMD:C_0603_1608Metric
- J2: footprint Connector_JST:JST_XH_B4B-XH-A_1x04_P2.50mm_Vertical -> Connector_PinSocket_2.54mm:PinSocket_1x04_P2.54mm_Vertical
- moved SW4 254.3 mm to (51.1, 159.4), turned to 90 degrees
- moved R9 252.8 mm to (52.2, 151.1), turned to -90 degrees
- moved C25 209.1 mm to (43.6, 114.8), turned to 180 degrees
- moved R6 206.1 mm to (44.0, 117.3), turned to 180 degrees
- moved D4 193.6 mm to (49.7, 116.0), turned to 180 degrees
- moved D5 180.2 mm to (69.6, 135.8)
- moved R7 168.9 mm to (75.8, 131.2), turned to 0 degrees
- moved C26 165.5 mm to (76.1, 133.2), turned to 180 degrees
- moved C24 145.1 mm to (137.1, 133.8)
- moved R5 141.0 mm to (137.0, 130.8)
- moved D3 137.8 mm to (143.4, 135.8)
- moved J3 130.7 mm to (70.2, 142.1)
- moved C5 123.1 mm to (115.8, 226.2), turned to 180 degrees
- moved C9 114.9 mm to (106.5, 226.2), turned to 180 degrees
- moved C6 111.5 mm to (103.1, 226.2), turned to 180 degrees
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Connections:
- net /CurrESC1 renamed /CurrESC1&2
Routing:
- net /TX: track 0.00 -> 3.36 mm, vias 0 -> 1
- net /RX: track 0.00 -> 3.24 mm, vias 0 -> 1
- net +3.3V: track 0.00 -> 3.03 mm, vias 0 -> 1
- net /CH340C/D-: track 88.3 -> 87.0 mm

Commit message: pcb changes
Parts:
- added ?: , clipboard:77f7410c-a6f3-441a-82db-5b2bc2281eba, F.Cu at (102.0, 254.4)
- added ?: , clipboard:77f7410c-a6f3-441a-82db-5b2bc2281eba, F.Cu at (107.0, 254.3)
- C10, C5, C6, C9, U2, U3: moved to F.Cu
- moved BZ1 116.3 mm to (134.2, 156.8), turned to 90 degrees
- moved R8 113.6 mm to (131.2, 139.4), turned to 180 degrees
- moved R4 113.0 mm to (142.9, 156.9), turned to 90 degrees
- moved Q1 109.3 mm to (133.1, 143.5)
- moved C25 71.6 mm to (112.6, 133.9), turned to 0 degrees
- moved R6 69.6 mm to (112.2, 131.3), turned to 0 degrees
- moved D4 59.3 mm to (106.6, 132.7), turned to 0 degrees
- moved C2 37.0 mm to (101.2, 197.2), turned to 180 degrees
- moved C28 36.8 mm to (112.4, 197.2), turned to 0 degrees
- moved C10 22.3 mm to (95.0, 203.8), turned to 0 degrees
- moved C5 22.3 mm to (117.0, 203.8), turned to 0 degrees
- moved C6 22.3 mm to (104.2, 203.8), turned to 0 degrees
- moved C9 22.3 mm to (107.6, 203.8), turned to 0 degrees
- moved J7 19.8 mm to (98.2, 224.8), turned to 0 degrees
- moved C16 19.0 mm to (142.2, 226.6), turned to -90 degrees
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Connections:
- R4 pad 2: /VM -> /Vb
Routing:
- net /CH340C/VMusC: track 16.7 -> 18.3 mm
- net Net-(BZ1-+): track 0.00 -> 1.01 mm

Commit message: PCB components order
Parts:
- removed ? (x2): , clipboard:77f7410c-a6f3-441a-82db-5b2bc2281eba
- removed C15: 10uF, Capacitor_Tantalum_SMD:CP_EIA-3216-10_Kemet-I_HandSolder
- removed C16, C25: 100nF, Capacitor_SMD:C_0805_2012Metric
- removed D4: WS2812B, LED_SMD:LED_WS2812B_PLCC4_5.0x5.0mm_P3.2mm
- removed J6: ESC1_VM, TerminalBlock_Phoenix:TerminalBlock_Phoenix_PT-1,5-2-3.5-H_1x02_P3.50mm_Horizontal
- removed J7: ESC2_VM, TerminalBlock_Phoenix:TerminalBlock_Phoenix_PT-1,5-2-3.5-H_1x02_P3.50mm_Horizontal
- removed J8: ESC3_VM, TerminalBlock_Phoenix:TerminalBlock_Phoenix_PT-1,5-2-3.5-H_1x02_P3.50mm_Horizontal
- removed R6: 100, Resistor_SMD:R_0805_2012Metric
- removed REF**: R_1206_3216Metric, Resistor_SMD:R_1206_3216Metric
- added J15: ESC_VM, TerminalBlock_Phoenix:TerminalBlock_Phoenix_PT-1,5-6-3.5-H_1x06_P3.50mm_Horizontal, F.Cu at (115.3, 234.6)
- C5, C6: footprint Capacitor_SMD:C_0805_2012Metric -> Capacitor_SMD:C_0603_1608Metric; moved to B.Cu
- J10, J11, J12: footprint Connector_JST:JST_XH_B2B-XH-A_1x02_P2.50mm_Vertical -> Connector_JST:JST_XH_S2B-XH-A_1x02_P2.50mm_Horizontal
- J17, J18, J19: footprint Connector_JST:JST_XH_B3B-XH-A_1x03_P2.50mm_Vertical -> MixLib:PinHeader_1x03_P2.54-SMD
- J3: footprint Connector_JST:JST_XH_B4B-XH-A_1x04_P2.50mm_Vertical -> Connector_PinSocket_2.54mm:PinSocket_1x04_P2.54mm_Vertical
- R10, R11, R12, R13: footprint Resistor_SMD:R_0805_2012Metric -> Resistor_SMD:R_0603_1608Metric
- U2, U3: moved to B.Cu
- moved R10 84.6 mm to (135.6, 236.9)
- moved R11 78.9 mm to (135.6, 235.2)
- moved R12 73.3 mm to (141.5, 226.8), turned to 180 degrees
- moved R13 71.7 mm to (141.5, 228.4), turned to 180 degrees
- moved R3 60.8 mm to (82.6, 145.2)
- moved D2 60.0 mm to (87.2, 224.9)
- moved R1 60.0 mm to (87.2, 226.8)
- moved C8 57.6 mm to (83.0, 143.2)
- moved C7 46.7 mm to (63.3, 173.4), turned to -90 degrees
- moved C28 38.5 mm to (122.6, 234.4), turned to 180 degrees
- moved C2 36.6 mm to (122.6, 226.9)
- moved R2 32.5 mm to (61.2, 173.6), turned to -90 degrees
- moved J19 31.0 mm to (157.2, 153.4)
- moved J18 30.5 mm to (151.2, 153.4)
- moved J17 30.2 mm to (145.2, 153.4)
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Connections:
- D5 pad 4: Net-(D4-DOUT) -> Net-(D3-DOUT)
- U1 pad 34: /RX -> /TX
- U1 pad 35: /TX -> /RX
Routing:
- net /Vb: track 0.00 -> 30.6 mm, vias 0 -> 3
- net +3.3V: track 3.03 -> 24.2 mm, vias 1 -> 2
- net /CH340C/CC2: track 0.00 -> 17.1 mm, vias 0 -> 2
- net /CH340C/CC1: track 0.00 -> 14.5 mm
- net /RX: track 3.24 -> 16.6 mm, vias 1 -> 2
- net /TX: track 3.36 -> 14.4 mm, vias 1 -> 2
- net /EN: track 0.00 -> 9.16 mm
- net Net-(U2-FILTER): track 0.00 -> 7.69 mm, vias 0 -> 1
- net /CH340C/D-: track 87.0 -> 94.7 mm, vias 0 -> 2
- net Net-(U3-FILTER): track 0.00 -> 7.46 mm, vias 0 -> 1
- net /SCL: track 0.00 -> 7.28 mm
- net /CH340C/VMusC: track 18.3 -> 25.5 mm, vias 0 -> 2
- net /SDA: track 0.00 -> 6.93 mm
- net /StepDown_2315/VCC_MP: track 0.00 -> 6.36 mm, vias 0 -> 1
- net Net-(ST1-EN/SYNC): track 0.00 -> 5.84 mm
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- added copper zone on F.Cu, net +3.3V
- added copper zone on F.Cu, net /StepDown_2315/BST
- added copper zone on F.Cu, net /StepDown_2315/FB
- added copper zone on F.Cu, net /StepDown_2315/Rt
- added copper zone on F.Cu, net /StepDown_2315/SW
- added copper zone on F.Cu, net /Vb
- added copper zone on B.Cu, net GND
- added copper zone on F.Cu, net GND
Other:
- outline, holes or cut-outs redrawn

Commit message: PCB advancements
Parts:
- added ESC_3: TerminalBlock_Phoenix_PT-1,5-3-3.5-H_1x03_P3.50mm_Horizontal, TerminalBlock_Phoenix:TerminalBlock_Phoenix_PT-1,5-3-3.5-H_1x03_P3.50mm_Horizontal, F.Cu at (110.0, 188.6)
- added H10: M2, MountingHole:MountingHole_2.2mm_M2, F.Cu at (109.7, 165.5)
- added H9: M2, MountingHole:MountingHole_2.2mm_M2, F.Cu at (103.3, 165.5)
- added REF**: R_1206_3216Metric, Resistor_SMD:R_1206_3216Metric, B.Cu at (69.4, 233.9)
- added REF**: R_1206_3216Metric, Resistor_SMD:R_1206_3216Metric, B.Cu at (143.8, 174.0)
- C22: value 22uF -> 10uF
- H7, H8: value M3 -> M2; footprint MountingHole:MountingHole_3mm -> MountingHole:MountingHole_2.2mm_M2
- moved H7 93.7 mm to (109.7, 159.2)
- moved H8 93.6 mm to (103.3, 159.2)
- moved R5 72.9 mm to (74.2, 133.2), turned to 90 degrees
- moved R7 70.8 mm to (138.7, 133.3)
- moved C26 70.8 mm to (136.7, 133.3)
- moved D3 70.3 mm to (70.8, 137.9), turned to 180 degrees
- moved D5 69.9 mm to (141.9, 137.7)
- moved C24 69.0 mm to (76.2, 133.2), turned to 90 degrees
- moved J17 29.2 mm to (174.3, 155.5), turned to 180 degrees
- moved J18 23.4 mm to (174.3, 149.4), turned to 180 degrees
- moved J19 19.8 mm to (174.3, 143.4), turned to 180 degrees
- moved SW2 13.2 mm to (68.6, 176.5), turned to -90 degrees
- moved J4 9.77 mm to (81.2, 177.5)
- moved J5 9.32 mm to (126.8, 178.0)
- moved C23 8.11 mm to (63.2, 230.8), turned to 90 degrees
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Connections:
- net /StepDown_2315/VCC_MP renamed /StepDown_2315/VCC_SW
- U1 pad 10: unconnected-(U1-IO25-Pad10) -> /ESC_3
- U1 pad 37: unconnected-(U1-IO23-Pad37) -> /LEDs
- U1 pad 4: unconnected-(U1-SENSOR_VP-Pad4) -> /CurrESC2
- U1 pad 5: unconnected-(U1-SENSOR_VN-Pad5) -> /CurrESC1&2
- U1 pad 6: unconnected-(U1-IO34-Pad6) -> /Enc1
- U1 pad 7: unconnected-(U1-IO35-Pad7) -> /Enc2
- U1 pad 8: unconnected-(U1-IO32-Pad8) -> /ESC_1
- U1 pad 9: unconnected-(U1-IO33-Pad9) -> /ESC_2
Routing:
- net /Vb: track 30.6 -> 116.8 mm, vias 3 -> 5
- net /ESC_3: track 0.00 -> 61.9 mm
- net /ESC_2: track 0.00 -> 55.4 mm
- net /ESC_1: track 0.00 -> 52.7 mm
- net /CH340C/VMusB: track 0.00 -> 17.7 mm, vias 0 -> 2
- net Net-(D1-A): track 0.00 -> 14.1 mm, vias 0 -> 1
- net /StepDown_2315/VCC_SW: track 6.36 -> 15.3 mm, vias 1 -> 2
- net +3.3V: track 24.2 -> 18.4 mm, vias 2 -> 3
- net /EN: track 9.16 -> 4.06 mm
- net Net-(D3-VDD): track 5.04 -> 0.00 mm
- net Net-(D5-VDD): track 4.72 -> 0.00 mm
- net /VM: track 0.00 -> 4.51 mm, vias 4 -> 12
- net GND: track 4.25 -> 0.00 mm, vias 8 -> 27
- net /CH340C/CC1: track 14.5 -> 17.0 mm
- net Net-(D2-K): track 0.00 -> 1.94 mm
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- added copper zone on B.Cu, net /ESC1&2_VM
- added copper zone on B.Cu, net /ESC3_VM
- added copper zone on B.Cu, net /VM
- added copper zone on F.Cu, net /VM
Other:
- board size 117.5 x 122 mm -> 109.5 x 122 mm

Commit message: pcb
Parts:
- removed J3: OLED, Connector_PinSocket_2.54mm:PinSocket_1x04_P2.54mm_Vertical
- J14: footprint Connector_JST:JST_XH_B4B-XH-A_1x04_P2.50mm_Vertical -> Connector_JST:JST_XH_S4B-XH-A_1x04_P2.50mm_Horizontal
- J2: footprint Connector_PinSocket_2.54mm:PinSocket_1x04_P2.54mm_Vertical -> MixLib:MPU6050_Module
- R4: footprint Resistor_SMD:R_0805_2012Metric -> Resistor_SMD:R_1206_3216Metric; moved to B.Cu
- moved C8 50.0 mm to (52.9, 174.7), turned to -90 degrees
- moved C7 43.6 mm to (91.0, 141.4), turned to 90 degrees
- moved R2 43.2 mm to (88.4, 141.7), turned to 90 degrees
- moved SW2 39.0 mm to (74.6, 137.9), turned to 0 degrees
- moved SW3 35.4 mm to (76.7, 178.4), turned to 0 degrees
- moved R9 32.3 mm to (85.2, 139.7)
- moved F1 26.7 mm to (65.4, 145.1)
- moved SW4 26.0 mm to (74.8, 143.7), turned to 180 degrees
- moved C3 23.0 mm to (64.1, 150.6)
- moved C4 17.1 mm to (64.1, 154.3)
- moved REF** 16.5 mm to (129.4, 165.8)
- moved J14 16.0 mm to (140.5, 158.1)
- moved D3 15.4 mm to (83.5, 129.1), turned to 90 degrees
- moved D5 15.1 mm to (129.5, 129.1), turned to 90 degrees
- moved U4 14.9 mm to (128.9, 169.5)
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Connections:
- net Net-(D3-DOUT) renamed /D_LED
- U1 pad 10: /ESC_3 -> unconnected-(U1-IO25-Pad10)
- U1 pad 37: /LEDs -> unconnected-(U1-IO23-Pad37)
- U1 pad 4: /CurrESC2 -> unconnected-(U1-SENSOR_VP-Pad4)
- U1 pad 5: /CurrESC1&2 -> unconnected-(U1-SENSOR_VN-Pad5)
- U1 pad 6: /Enc1 -> unconnected-(U1-IO34-Pad6)
- U1 pad 7: /Enc2 -> unconnected-(U1-IO35-Pad7)
- U1 pad 8: /ESC_1 -> unconnected-(U1-IO32-Pad8)
- U1 pad 9: /ESC_2 -> unconnected-(U1-IO33-Pad9)
Routing:
- net /ESC_3: track 61.9 -> 0.00 mm
- net /ESC_2: track 55.4 -> 0.00 mm
- net /ESC_1: track 52.7 -> 0.00 mm
- net +3.3V: track 18.4 -> 37.2 mm, vias 3 -> 4
- net /Vb: track 116.8 -> 131.4 mm
- net /CH340C/D+: track 83.6 -> 96.9 mm
- net /VDD_ESP: track 0.00 -> 12.2 mm
- net /TX: track 14.5 -> 6.17 mm, vias 2 -> 1
- net /RX: track 16.8 -> 8.56 mm, vias 2 -> 1
- net /SCL: track 7.28 -> 0.00 mm
- net /SDA: track 6.93 -> 0.00 mm
- net /CH340C/D-: track 94.7 -> 99.1 mm
- net /EN: track 4.06 -> 0.00 mm
- net Net-(BZ1-+): track 1.01 -> 0.00 mm
Other:
- board size 109.5 x 122 mm -> 89 x 122 mm
- board text removed: "puedo mover conector mas adelante"
