File: pcb/main_MagicAlonso/main_MagicAlonso.kicad_pcb (KiCad board)
At the start: 2 copper layers, 89 x 122 mm, 91 parts, among them J1 XT30PW-M, J10 ESC1, J11 ESC2, J12 ESC3, J13 USB_C_Receptacle_USB2.0_16P, J14 UART_Out, J15 ESC_VM, J16 USB_B_Micro, J17 aux0, J18 aux2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

Commit message: mais avances en la pcb
Parts:
- C8: footprint Capacitor_SMD:C_0805_2012Metric -> Capacitor_SMD:C_0603_1608Metric
- moved R3 39.6 mm to (97.1, 185.6)
- moved C8 34.2 mm to (87.0, 174.7)
- moved C7 17.4 mm to (108.4, 142.0)
- moved R2 17.4 mm to (105.8, 142.2)
- moved R9 17.4 mm to (102.6, 140.3)
- moved SW4 8.53 mm to (83.3, 144.0), turned to -90 degrees
- moved SW2 6.26 mm to (73.2, 144.0), turned to -90 degrees
- moved R1 5.32 mm to (95.0, 225.5), turned to 0 degrees
- moved SW3 4.10 mm to (72.6, 178.3), turned to 180 degrees
- moved J10 1.18 mm to (97.4, 197.3)
- moved J11 1.18 mm to (105.2, 197.3)
- moved J12 1.18 mm to (113.0, 197.3)
- moved F1 1.04 mm to (66.4, 145.3)
- moved C3 0.77 mm to (64.1, 151.3)
- moved C4 0.77 mm to (64.1, 155.0)
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Connections:
- U1 pad 14: unconnected-(U1-IO12-Pad14) -> /ESC_1
- U1 pad 16: unconnected-(U1-IO13-Pad16) -> /ESC_2
- U1 pad 23: unconnected-(U1-IO15-Pad23) -> /ESC_3
- U1 pad 26: unconnected-(U1-IO4-Pad26) -> /Enc1
- U1 pad 27: unconnected-(U1-IO16-Pad27) -> /Enc2
- U1 pad 4: unconnected-(U1-SENSOR_VP-Pad4) -> /BUTTON
Routing:
- net +3.3V: track 37.2 -> 112.1 mm, vias 4 -> 3
- net /ESC_1: track 0.00 -> 52.0 mm
- net /ESC_3: track 0.00 -> 49.0 mm
- net /ESC_2: track 0.00 -> 47.9 mm
- net /Enc2: track 0.00 -> 46.3 mm
- net /BUTTON: track 0.00 -> 30.3 mm, vias 0 -> 2
- net /EN: track 0.00 -> 22.4 mm, vias 0 -> 2
- net /BOOT: track 0.00 -> 15.3 mm, vias 0 -> 1
- net /Enc1: track 0.00 -> 10.7 mm
- net /VDD_ESP: track 12.2 -> 13.6 mm
- net /StepDown_2315/VCC_SW: track 15.3 -> 16.4 mm
- net /Vb: track 131.4 -> 132.6 mm
- net Net-(D2-K): track 1.94 -> 3.01 mm
- net GND: vias 27 -> 28

Commit message: Update PCB
Parts:
- R3: moved to B.Cu
- R4: moved to F.Cu
- moved REF** 26.1 mm to (155.2, 161.8)
- moved R3 16.0 mm to (86.2, 173.8), turned to 90 degrees
- moved R8 15.4 mm to (124.2, 141.9), turned to -90 degrees
- moved R5 11.8 mm to (89.2, 137.1), turned to 0 degrees
- moved C24 11.8 mm to (89.1, 135.2), turned to 0 degrees
- moved Q1 10.3 mm to (130.2, 141.8)
- moved C11 10.2 mm to (96.4, 143.2)
- moved C12 9.84 mm to (96.7, 139.8)
- moved J9 8.47 mm to (117.8, 134.1)
- moved C26 7.97 mm to (137.7, 136.9)
- moved R7 7.97 mm to (137.7, 138.9)
- moved R4 7.86 mm to (141.3, 144.2), turned to 180 degrees
- moved H5 7.54 mm to (89.0, 130.7)
- moved H6 7.54 mm to (124.0, 130.7)
- moved D3 6.57 mm to (82.6, 135.6), turned to 180 degrees
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Routing:
- net /SDA: track 0.00 -> 69.2 mm, vias 0 -> 1
- net +3.3V: track 112.1 -> 80.2 mm
- net /Vb: track 132.6 -> 119.3 mm
- net /Enc1: track 10.7 -> 20.1 mm, vias 0 -> 1
- net /SCL: track 0.00 -> 6.34 mm, vias 0 -> 1
- net /CH340C/D-: track 99.1 -> 105.2 mm
- net Net-(D5-VDD): track 0.00 -> 5.93 mm
- net /BOOT: track 15.3 -> 20.5 mm
- net Net-(D3-VDD): track 0.00 -> 5.22 mm
- net /D_LED: track 0.00 -> 3.78 mm, vias 0 -> 1
- net /CH340C/VMusB: track 17.2 -> 14.8 mm
- net /RX: track 8.56 -> 6.22 mm
- net Net-(U2-FILTER): track 7.69 -> 9.93 mm
- net Net-(U3-FILTER): track 7.46 -> 9.59 mm
- net /VDD_ESP: track 13.6 -> 15.2 mm
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Other:
- board size 89 x 122 mm -> 89 x 113.2 mm
- board text added: "EN"
- board text added: "PUSH"

Commit message: update PCB
Parts:
- REF**: moved to F.Cu
- moved R2 24.3 mm to (87.5, 142.4), turned to 0 degrees
- moved R9 21.7 mm to (87.9, 150.6), turned to 90 degrees
- moved REF** 15.2 mm to (141.8, 168.9)
- moved SW2 14.5 mm to (87.6, 145.6), turned to 0 degrees
- moved D7 14.2 mm to (144.8, 178.6)
- moved SW4 7.68 mm to (75.8, 145.6), turned to 0 degrees
- moved C11 5.42 mm to (92.8, 139.2), turned to 90 degrees
- moved J14 4.41 mm to (140.5, 162.8)
- moved J2 2.66 mm to (136.7, 155.8)
- moved C9 1.48 mm to (116.1, 224.5)
- moved C12 1.40 mm to (95.4, 139.2), turned to 90 degrees
- moved C3 1.04 mm to (64.1, 152.3)
- moved C5 0.71 mm to (123.7, 226.1)
- moved D2 0.68 mm to (90.8, 225.0)
- moved R1 0.68 mm to (95.5, 225.1)
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Connections:
- REF** pad 1: /Vb -> /CH340C/D-
- REF** pad 2: /Vb -> /CH340C/D-
- U1 pad 12: unconnected-(U1-IO27-Pad12) -> /CurrESC2
- U1 pad 13: unconnected-(U1-IO14-Pad13) -> /CurrESC1&2
- U1 pad 30: unconnected-(U1-IO18-Pad30) -> /Data_2aux
- U1 pad 31: unconnected-(U1-IO19-Pad31) -> /Data_1aux
- U1 pad 37: unconnected-(U1-IO23-Pad37) -> /Data_0aux
Routing:
- net /CurrESC1&2: track 0.00 -> 104.0 mm, vias 0 -> 1
- net /CurrESC2: track 0.00 -> 98.6 mm, vias 0 -> 1
- net +3.3V: track 80.2 -> 173.2 mm, vias 3 -> 4
- net /SCL: track 6.34 -> 75.1 mm
- net /TX: track 5.17 -> 24.4 mm
- net /Vb: track 119.3 -> 101.0 mm
- net /EN: track 23.2 -> 38.2 mm
- net /BUTTON: track 29.1 -> 40.1 mm
- net /RX: track 6.22 -> 15.7 mm
- net /CH340C/VMusB: track 14.8 -> 6.13 mm, vias 2 -> 0
- net /Enc1: track 20.1 -> 11.8 mm, vias 1 -> 0
- net /CH340C/D-: track 105.2 -> 100.7 mm, vias 2 -> 0
- net Net-(U3-FILTER): track 9.59 -> 12.9 mm
- net Net-(U2-FILTER): track 9.93 -> 11.8 mm
- net /CH340C/D+: track 96.4 -> 97.5 mm
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Other:
- board text added: "Testear resistencias 0ohms"
- board text removed: "EN"
- board text removed: "PUSH"

Commit message: Update PCB
Parts:
- moved C7 27.3 mm to (87.9, 147.9), turned to 0 degrees
- moved R9 13.9 mm to (74.4, 147.5), turned to 0 degrees
- moved R3 4.74 mm to (89.0, 177.6), turned to 0 degrees
- moved R2 3.83 mm to (87.6, 146.2)
- moved C8 2.41 mm to (89.4, 175.4), turned to 180 degrees
- moved SW2 2.39 mm to (86.9, 143.3)
- moved SW4 2.28 mm to (75.8, 143.3)
- moved C9 1.85 mm to (114.2, 224.4)
- moved D2 1.60 mm to (89.2, 225.0)
- moved R1 1.60 mm to (93.8, 225.1)
- moved C4 1.04 mm to (64.5, 154.1)
- moved C3 1.04 mm to (64.4, 151.4)
- moved C11 0.32 mm to (92.5, 139.1)
- moved C12 0.32 mm to (95.1, 139.1)
Connections:
- U1 pad 26: /Enc1 -> /BUZ
- U1 pad 27: /Enc2 -> /Data_S3
- U1 pad 28: unconnected-(U1-IO17-Pad28) -> /Data_S2
- U1 pad 30: /Data_2aux -> /Data_S1
- U1 pad 31: /Data_1aux -> /Data_S0
- U1 pad 5: unconnected-(U1-SENSOR_VN-Pad5) -> /Enc2
- U1 pad 6: unconnected-(U1-IO34-Pad6) -> /Enc1
Routing:
- net +3.3V: track 173.2 -> 383.6 mm, vias 4 -> 5
- net /Data_S3: track 0.00 -> 88.1 mm
- net /Data_S2: track 0.00 -> 84.4 mm
- net /RX: track 15.7 -> 97.8 mm, vias 1 -> 2
- net /TX: track 24.4 -> 91.4 mm, vias 1 -> 2
- net /Data_S1: track 0.00 -> 44.3 mm
- net /Data_S0: track 0.00 -> 41.1 mm
- net /Enc1: track 11.8 -> 48.3 mm, vias 0 -> 1
- net /Enc2: track 46.3 -> 81.6 mm, vias 0 -> 1
- net /Data_0aux: track 0.00 -> 32.3 mm
- net /EN: track 38.2 -> 43.7 mm
- net /BUTTON: track 40.1 -> 34.9 mm
- net /BOOT: track 20.5 -> 25.2 mm
- net /SCL: track 75.1 -> 77.0 mm
- net /SDA: track 68.3 -> 70.0 mm
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Other:
- outline, holes or cut-outs redrawn

Commit message: first PCB layout done
Parts:
- removed J17: aux0, MixLib:PinHeader_1x03_P2.54-SMD
- removed J18: aux2, MixLib:PinHeader_1x03_P2.54-SMD
- removed J19: aux1, MixLib:PinHeader_1x03_P2.54-SMD
- added ?: , , F.Cu at (97.7, 210.9)
- added ?: , , F.Cu at (122.0, 141.1)
- added ?: , , F.Cu at (122.0, 139.0)
- added ?: , , F.Cu at (133.8, 178.8)
- added ?: , , F.Cu at (149.6, 226.9)
- added ?: , , F.Cu at (63.7, 148.6)
- added ?: , , F.Cu at (106.5, 210.9)
- added ?: , , F.Cu at (115.3, 210.9)
- added ?: , , F.Cu at (73.3, 137.8)
- added ?: , , F.Cu at (133.8, 180.8)
- added R6: 10k, Resistor_SMD:R_0805_2012Metric, F.Cu at (94.9, 142.6)
- added REF**: MagicAlonso_Red_Mod_23.5mm, MixLib:MagicAlonso_Red_Mod_23.5mm, F.Cu at (135.3, 206.2)
- added REF**: MagicAlonso_Red_Mod_23.5mm, MixLib:MagicAlonso_Red_Mod_23.5mm, F.Cu at (77.8, 200.4)
- moved R4 3.73 mm to (143.0, 147.6), turned to 0 degrees
- moved R9 3.63 mm to (70.8, 147.7)
- moved R8 2.69 mm to (123.7, 144.6)
- moved F1 1.59 mm to (66.7, 145.1)
- moved Q1 1.39 mm to (128.8, 141.8)
- moved C13 1.21 mm to (138.8, 173.4)
- moved C14 1.21 mm to (138.6, 171.6)
- moved C8 1.02 mm to (90.2, 174.8), turned to -90 degrees
- moved J14 1.00 mm to (141.5, 162.8)
- moved C7 1.00 mm to (86.9, 147.9)
- moved R2 0.99 mm to (86.7, 146.2)
- moved R3 0.64 mm to (88.4, 177.7)
- moved C24 0.62 mm to (89.1, 135.8)
- moved R5 0.62 mm to (89.2, 137.8)
Connections:
- net /Data_0aux renamed /Data_EN
- U1 pad 10: unconnected-(U1-IO25-Pad10) -> /Enc2
- U1 pad 11: unconnected-(U1-IO26-Pad11) -> /Enc1
- U1 pad 26: /BUZ -> unconnected-(U1-IO4-Pad26)
- U1 pad 5: /Enc2 -> /Data_SIG
- U1 pad 6: /Enc1 -> unconnected-(U1-IO34-Pad6)
- U1 pad 7: unconnected-(U1-IO35-Pad7) -> /Data_1aux
- U1 pad 8: unconnected-(U1-IO32-Pad8) -> /Data_2aux
- U1 pad 9: unconnected-(U1-IO33-Pad9) -> /BUZ
Routing:
- net /Vb: track 101.0 -> 194.3 mm, vias 5 -> 7
- net /BUZ: track 0.00 -> 78.8 mm, vias 0 -> 2
- net /Data_2aux: track 0.00 -> 76.0 mm, vias 0 -> 1
- net /Data_1aux: track 0.00 -> 71.8 mm, vias 0 -> 1
- net /Data_SIG: track 0.00 -> 67.5 mm, vias 0 -> 1
- net +3.3V: track 383.6 -> 439.9 mm, vias 5 -> 7
- net /D_LED: track 3.78 -> 47.3 mm, vias 1 -> 0
- net /VM: track 4.51 -> 25.0 mm
- net Net-(BZ1--): track 0.00 -> 12.9 mm, vias 0 -> 1
- net /Enc1: track 48.3 -> 37.8 mm
- net Net-(BZ1-+): track 0.00 -> 9.12 mm, vias 0 -> 1
- net /Enc2: track 81.6 -> 74.9 mm
- net /SCL: track 77.0 -> 70.9 mm
- net Net-(Q1-G): track 0.00 -> 6.02 mm
- net Net-(U3-FILTER): track 12.9 -> 9.91 mm
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Other:
- outline, holes or cut-outs redrawn
- board text removed: "Testear resistencias 0ohms"
