File: pcb/main_MagicAlonso/rounded/main_MagicAlonso-rounded.kicad_pcb (KiCad board)
At the start: 2 copper layers, 89 x 113.2 mm, 103 parts, among them J1 XT30PW-M, J10 ESC1, J11 ESC2, J12 ESC3, J13 USB_C_Receptacle_USB2.0_16P, J14 UART_Out, J15 ESC_VM, J16 USB_B_Micro, J2 MPU6050, J4 Encoder1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

Commit message: sensors pcb update
Routing:
- net /BOOT: track 25.2 -> 24.5 mm
