File: pcb/sensors16_MagicAlonso/sensors16_MagicAlonso.kicad_sch (KiCad schematic)
At the start: 55 parts, among them J9 Sensors, U1 QRE1113GR, U10 QRE1113GR, U11 QRE1113GR, U12 QRE1113GR, U13 QRE1113GR, U14 QRE1113GR, U15 QRE1113GR, U16 QRE1113GR, U17 CD74HC4067, U18 CD74HC4067M, U2 QRE1113GR, U3 QRE1113GR, U4 QRE1113GR, U5 QRE1113GR, U6 QRE1113GR, U7 QRE1113GR, U8 QRE1113GR, U9 QRE1113GR

Commit message: pcb update
Parts:
- added C24, C26: 100nF, Capacitor_SMD:C_0805_2012Metric, symbol Device:C_Small
- added D3, D5: WS2812B, LED_SMD:LED_WS2812B_PLCC4_5.0x5.0mm_P3.2mm, symbol LED:WS2812B
- added R33: 10k, symbol Device:R_Small
- added R34, R35: 100, Resistor_SMD:R_0805_2012Metric, symbol Device:R_Small
Connections:
- net +3.3V: now also R34.2, R35.2
- net GND: now also C24.2, C26.2, D3.3 (VSS), D5.3 (VSS), R33.2
- net EN: now reaches U17.22 (~{EN})
- net EN: now also U18.15 (~{E}), R33.1
- net Data_1aux renamed LEDs
- net LEDs: now also D3.4 (DIN)
- new net: C24.1, D3.1 (VDD), R34.1
- new net: C26.1, D5.1 (VDD), R35.1
- new net D_LED: D3.2 (DOUT), D5.4 (DIN)
Other:
- note added: "LEDs"
- moved on the sheet: C11, C12, J9, R1, R10, R11, R12, R13, R14, R15, R16, R17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

Commit message: sensors pcb update
Parts:
- added H1, H2: MountingHole, MountingHole:MountingHole_3.2mm_M3_DIN965, symbol Mechanical:MountingHole
- C1, C2: footprint (none) -> Capacitor_SMD:C_0805_2012Metric
- R1: renamed from R17; footprint EESTN5-v2:R_0805 -> Resistor_SMD:R_0805_2012Metric
- R10: renamed from R21; footprint EESTN5-v2:R_0805 -> Resistor_SMD:R_0805_2012Metric
- R11: renamed from R3; footprint EESTN5-v2:R_0805 -> Resistor_SMD:R_0805_2012Metric
- R12: renamed from R4; footprint EESTN5-v2:R_0805 -> Resistor_SMD:R_0805_2012Metric
- R13: renamed from R20; footprint EESTN5-v2:R_0805 -> Resistor_SMD:R_0805_2012Metric
- R14: renamed from R23; footprint EESTN5-v2:R_0805 -> Resistor_SMD:R_0805_2012Metric
- R15: renamed from R7; footprint EESTN5-v2:R_0805 -> Resistor_SMD:R_0805_2012Metric
- R16: renamed from R8; footprint EESTN5-v2:R_0805 -> Resistor_SMD:R_0805_2012Metric
- R17: renamed from R22; footprint EESTN5-v2:R_0805 -> Resistor_SMD:R_0805_2012Metric
- R18: renamed from R25; footprint EESTN5-v2:R_0805 -> Resistor_SMD:R_0805_2012Metric
- R19: renamed from R9; footprint EESTN5-v2:R_0805 -> Resistor_SMD:R_0805_2012Metric
- R2: renamed from R30; footprint EESTN5-v2:R_0805 -> Resistor_SMD:R_0805_2012Metric
- R20: renamed from R10; footprint EESTN5-v2:R_0805 -> Resistor_SMD:R_0805_2012Metric
- R21: renamed from R33; footprint (none) -> Resistor_SMD:R_0805_2012Metric
- R22: renamed from R24; footprint EESTN5-v2:R_0805 -> Resistor_SMD:R_0805_2012Metric
- R23: renamed from R27; footprint EESTN5-v2:R_0805 -> Resistor_SMD:R_0805_2012Metric
- R24: renamed from R11; footprint EESTN5-v2:R_0805 -> Resistor_SMD:R_0805_2012Metric
- R25: renamed from R12; footprint EESTN5-v2:R_0805 -> Resistor_SMD:R_0805_2012Metric
- R26, R31: footprint EESTN5-v2:R_0805 -> Resistor_SMD:R_0805_2012Metric
- R27: renamed from R29; footprint EESTN5-v2:R_0805 -> Resistor_SMD:R_0805_2012Metric
- R28: renamed from R13; footprint EESTN5-v2:R_0805 -> Resistor_SMD:R_0805_2012Metric
- R29: renamed from R14; footprint EESTN5-v2:R_0805 -> Resistor_SMD:R_0805_2012Metric
- R3: renamed from R1; footprint EESTN5-v2:R_0805 -> Resistor_SMD:R_0805_2012Metric
- R30: renamed from R28; footprint EESTN5-v2:R_0805 -> Resistor_SMD:R_0805_2012Metric
- R32: renamed from R15; footprint EESTN5-v2:R_0805 -> Resistor_SMD:R_0805_2012Metric
- R33: renamed from R16; footprint EESTN5-v2:R_0805 -> Resistor_SMD:R_0805_2012Metric
- R4: renamed from R2; footprint EESTN5-v2:R_0805 -> Resistor_SMD:R_0805_2012Metric
- R5: renamed from R19; footprint EESTN5-v2:R_0805 -> Resistor_SMD:R_0805_2012Metric
- R6: renamed from R32; footprint EESTN5-v2:R_0805 -> Resistor_SMD:R_0805_2012Metric
- R7: renamed from R5; footprint EESTN5-v2:R_0805 -> Resistor_SMD:R_0805_2012Metric
- R8: renamed from R6; footprint EESTN5-v2:R_0805 -> Resistor_SMD:R_0805_2012Metric
- R9: renamed from R18; footprint EESTN5-v2:R_0805 -> Resistor_SMD:R_0805_2012Metric
- renumbered C12 to C3, C24 to C4, C11 to C5, C26 to C6, D3 to D1, D5 to D2, J9 to J1, U9 to U1, U13 to U10, U5 to U11, U6 to U12, U14 to U13, U15 to U14, U7 to U15, U8 to U16, U16 to U2, U17 to U20, U1 to U3, U18 to U30, U2 to U4, U10 to U5, U11 to U6, U3 to U7, U4 to U8, U12 to U9
Other:
- moved on the sheet: R1, R2, R3, R4, R5, R6, R7, R8, U1, U2, U3, U4

Commit message: sensors16 pcb update
Parts:
- renumbered C1 to C0, C2 to C1, C3 to C2, C4 to C3, C5 to C4, C6 to C5, D1 to D0, D2 to D1, J1 to J0, U30 to M0, U20 to M1, R2 to R0, R3 to R1, R12 to R10, R10 to R11, R13 to R12, R15 to R13, R16 to R14, R14 to R15, R17 to R16, R19 to R17, R20 to R18, R18 to R19, R4 to R2, R22 to R20, R24 to R22, R25 to R23, R23 to R24, R26 to R25, R28 to R26, R29 to R27, R27 to R28, R30 to R29, R1 to R3, R32 to R30, R33 to R31, R31 to R32, R34 to R33, R35 to R34, R6 to R4, R7 to R5, R8 to R6, R5 to R7, R9 to R8, R11 to R9, U2 to U0, U3 to U1, U12 to U10, U10 to U11, U13 to U12, U15 to U13, U16 to U14, U14 to U15, U4 to U2, U1 to U3, U5 to U4, U7 to U5, U8 to U6, U6 to U7, U9 to U8, U11 to U9
Other:
- moved on the sheet: R11, R12, R13, R15, R16, R17, R18, R2, R20, R22, R23, R25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
