File: pcb/sensors16_MagicAlonso/sensors16_MagicAlonso.kicad_pcb (KiCad board)
At the start: 2 copper layers, 64 parts, among them J1 Sensors, U1 QRE1113GR, U10 QRE1113GR, U11 QRE1113GR, U12 QRE1113GR, U13 QRE1113GR, U14 QRE1113GR, U15 QRE1113GR, U16 QRE1113GR, U2 QRE1113GR, U20 CD74HC4067, U3 QRE1113GR, U30 CD74HC4067M, U4 QRE1113GR, U5 QRE1113GR, U6 QRE1113GR, U7 QRE1113GR, U8 QRE1113GR, U9 QRE1113GR

Commit message: sensors16 pcb update
Parts:
- removed U16: QRE1113GR, OptoDevice:OnSemi_CASE100CY
- removed U20: CD74HC4067, MixLib:CD74HC4067_module
- added M1: CD74HC4067, MixLib:CD74HC4067_module, F.Cu at (252.8, 131.1)
- added U0: QRE1113GR, OptoDevice:OnSemi_CASE100CY, F.Cu at (24.1, 153.0)
- U10, U11, U12, U13, U14, U15, U9: moved to F.Cu
- moved U6 100.2 mm to (60.1, 153.0)
- moved U3 87.9 mm to (42.1, 153.0)
- moved U1 86.3 mm to (30.1, 153.0)
- moved U2 79.5 mm to (36.1, 153.0)
- moved U5 73.6 mm to (54.1, 153.0)
- moved U4 69.0 mm to (48.1, 153.0)
- moved U7 61.0 mm to (66.1, 153.0)
- moved U8 60.4 mm to (72.1, 153.0)
- moved U10 52.2 mm to (84.1, 153.0), turned to 0 degrees
- moved U11 50.2 mm to (90.1, 153.0), turned to 0 degrees
- moved U9 45.3 mm to (78.1, 153.0), turned to 0 degrees
- moved U12 40.5 mm to (96.1, 153.0), turned to 0 degrees
- moved U13 29.6 mm to (102.1, 153.0), turned to 0 degrees
- moved U15 23.8 mm to (114.1, 153.0), turned to 0 degrees
- moved U14 19.1 mm to (108.1, 153.0), turned to 0 degrees
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- renumbered C1 to C0, C2 to C1, C3 to C2, C4 to C3, C5 to C4, C6 to C5, D1 to D0, D2 to D1, J1 to J0, U30 to M0, R2 to R0, R3 to R1, R12 to R10, R10 to R11, R13 to R12, R15 to R13, R16 to R14, R14 to R15, R17 to R16, R19 to R17, R20 to R18, R18 to R19, R4 to R2, R22 to R20, R24 to R22, R25 to R23, R23 to R24, R26 to R25, R28 to R26, R29 to R27, R27 to R28, R30 to R29, R1 to R3, R32 to R30, R33 to R31, R31 to R32, R34 to R33, R35 to R34, R6 to R4, R7 to R5, R8 to R6, R5 to R7, R9 to R8, R11 to R9
Connections:
- R0 pad 2: Net-(U2-A) -> Net-(U0-A)
- R1 pad 2: Net-(U3-A) -> Net-(U1-A)
- R10 pad 2: Net-(U8-A) -> Net-(U6-A)
- R11 pad 2: Net-(U6-A) -> Net-(U7-A)
- R16 pad 2: Net-(U9-A) -> Net-(U8-A)
- R17 pad 2: Net-(U11-A) -> Net-(U9-A)
- R18 pad 2: Net-(U12-A) -> Net-(U10-A)
- R19 pad 2: Net-(U10-A) -> Net-(U11-A)
- R2 pad 2: Net-(U4-A) -> Net-(U2-A)
- R25 pad 2: Net-(U13-A) -> Net-(U12-A)
- R26 pad 2: Net-(U15-A) -> Net-(U13-A)
- R27 pad 2: Net-(U16-A) -> Net-(U14-A)
- R28 pad 2: Net-(U14-A) -> Net-(U15-A)
- R3 pad 2: Net-(U1-A) -> Net-(U3-A)
- R8 pad 2: Net-(U5-A) -> Net-(U4-A)
- R9 pad 2: Net-(U7-A) -> Net-(U5-A)
- U1 pad 3: /QRE_3 -> /QRE_1
- U10 pad 3: /QRE_11 -> /QRE_10
- U11 pad 3: /QRE_9 -> /QRE_11
- U12 pad 3: /QRE_10 -> /QRE_12
- U13 pad 3: /QRE_12 -> /QRE_13
- U14 pad 3: /QRE_15 -> /QRE_14
- U15 pad 3: /QRE_13 -> /QRE_15
- U2 pad 3: /QRE_0 -> /QRE_2
- U3 pad 3: /QRE_1 -> /QRE_3
- U4 pad 3: /QRE_2 -> /QRE_4
- U5 pad 3: /QRE_4 -> /QRE_5
- U6 pad 3: /QRE_7 -> /QRE_6
- U7 pad 3: /QRE_5 -> /QRE_7
- U8 pad 3: /QRE_6 -> /QRE_8
- U9 pad 3: /QRE_8 -> /QRE_9

Commit message: sensors pcb update
Parts:
- U0, U1, U10, U11, U12, U13, U14, U15, U2, U3, U4, U5, U6, U7, U8, U9: moved to B.Cu
- moved U10 115.4 mm to (166.8, 72.5), turned to 180 degrees
- moved U9 115.4 mm to (159.8, 71.5), turned to 180 degrees
- moved U11 115.1 mm to (173.8, 74.0), turned to 180 degrees
- moved U8 115.0 mm to (152.8, 71.2), turned to 180 degrees
- moved U12 114.3 mm to (180.8, 76.2), turned to 180 degrees
- moved U7 114.3 mm to (145.8, 71.2), turned to 180 degrees
- moved U6 113.3 mm to (138.8, 71.5), turned to 180 degrees
- moved U13 113.2 mm to (187.8, 79.0), turned to 180 degrees
- moved U5 111.9 mm to (131.8, 72.5), turned to 180 degrees
- moved U14 111.7 mm to (194.8, 82.5), turned to 180 degrees
- moved U4 110.1 mm to (124.8, 74.0), turned to 180 degrees
- moved U15 109.9 mm to (201.8, 86.8), turned to 180 degrees
- moved U3 107.8 mm to (117.8, 76.2), turned to 180 degrees
- moved U2 105.1 mm to (110.8, 79.0), turned to 180 degrees
- moved U1 102.0 mm to (103.8, 82.5), turned to 180 degrees
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Other:
- board outline added: 140 x 28.6 mm
