File: pcb/main_Magic-simple/StepDown_2315.kicad_sch (KiCad schematic)
At the start: 19 parts, among them U5 CN3903, U6 Mini360

Commit message: pcbAAAAA
Parts:
- removed U5: CN3903, Package_SO:SOIC-8-1EP_3.9x4.9mm_P1.27mm_EP2.41x3.3mm, symbol MixLib:CN3903
Changed lines of the file:
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@@
 		)
 		(instances
-			(project "main_MagicAlonso__test"
+			(project "main_MagicAlonso"
 				(path "/80af5e1a-3060-4775-9fc3-f6762d1535e7/38d4c26b-5042-47e6-b450-9f4e66fb3158"
 					(reference "#PWR060")
@@
 		)
 		(instances
-			(project "main_MagicAlonso__test"
+			(project "main_MagicAlonso"
 				(path "/80af5e1a-3060-4775-9fc3-f6762d1535e7/38d4c26b-5042-47e6-b450-9f4e66fb3158"
 					(reference "Rp1")
@@
 		)
 		(instances
-			(project "main_MagicAlonso__test"
+			(project "main_MagicAlonso"
 				(path "/80af5e1a-3060-4775-9fc3-f6762d1535e7/38d4c26b-5042-47e6-b450-9f4e66fb3158"
 					(reference "R15")
@@
 		)
 		(instances
-			(project "main_MagicAlonso__test"
+			(project "main_MagicAlonso"
 				(path "/80af5e1a-3060-4775-9fc3-f6762d1535e7/38d4c26b-5042-47e6-b450-9f4e66fb3158"
 					(reference "R14")
@@
 		)
 		(instances
-			(project "main_MagicAlonso__test"
+			(project "main_MagicAlonso"
 				(path "/80af5e1a-3060-4775-9fc3-f6762d1535e7/38d4c26b-5042-47e6-b450-9f4e66fb3158"
 					(reference "C20")
-					(unit 1)
-				)
-			)
-		)
-	)
-	(symbol
-		(lib_id "MixLib:CN3903")
-		(at 181.61 49.53 0)
-		(unit 1)
-		(exclude_from_sim no)
-		(in_bom yes)
-		(on_board yes)
-		(dnp no)
-		(fields_autoplaced yes)
-		(property "Reference" "U5"
-			(at 183.7533 33.02 0)
-			(effects
-				(font
-					(size 1.27 1.27)
-				)
-				(justify left)
-			)
-		)
-		(property "Value" "CN3903"
-			(at 183.7533 35.56 0)
-			(effects
-				(font
-					(size 1.27 1.27)
-				)
-				(justify left)
-			)
-		)
-		(property "Footprint" "Package_SO:SOIC-8-1EP_3.9x4.9mm_P1.27mm_EP2.41x3.3mm"
-			(at 183.642 83.312 0)
-			(effects
-				(font
-					(size 1.27 1.27)
-				)
-				(hide yes)
-			)
-		)
-		(property "Datasheet" "https://datasheet4u.com/pdf-down/C/N/3/CN3903-Chipnet.pdf"
-			(at 183.896 78.994 0)
-			(effects
-				(font
-					(size 1.27 1.27)
-				)
-				(hide yes)
-			)
-		)
-		(property "Description" "36V 3.5A 500KHz Synchronous Step-Down Converter"
-			(at 183.134 75.184 0)
-			(effects
-				(font
-					(size 1.27 1.27)
-				)
-				(hide yes)
-			)
-		)
-		(pin "8"
-		)
-		(pin "4"
-		)
-		(pin "5"
-		)
-		(pin "1"
-		)
-		(pin "2"
-		)
-		(pin "6"
-		)
-		(pin "3"
-		)
-		(pin "9"
-		)
-		(pin "7"
-		)
-		(instances
-			(project ""
-				(path "/80af5e1a-3060-4775-9fc3-f6762d1535e7/38d4c26b-5042-47e6-b450-9f4e66fb3158"
-					(reference "U5")
 					(unit 1)
 				)
@@
 		)
 		(instances
-			(project "main_MagicAlonso__test"
+			(project ""
 				(path "/80af5e1a-3060-4775-9fc3-f6762d1535e7/38d4c26b-5042-47e6-b450-9f4e66fb3158"
 					(reference "Rt1")
@@
 		)
 		(instances
-			(project "main_MagicAlonso__test"
+			(project ""
 				(path "/80af5e1a-3060-4775-9fc3-f6762d1535e7/38d4c26b-5042-47e6-b450-9f4e66fb3158"
 					(reference "#PWR056")
@@
 		)
 		(instances
-			(project "main_MagicAlonso__test"
+			(project "main_MagicAlonso"
 				(path "/80af5e1a-3060-4775-9fc3-f6762d1535e7/38d4c26b-5042-47e6-b450-9f4e66fb3158"
 					(reference "C23")
@@
 		)
 		(instances
-			(project "main_MagicAlonso__test"
+			(project "main_MagicAlonso"
 				(path "/80af5e1a-3060-4775-9fc3-f6762d1535e7/38d4c26b-5042-47e6-b450-9f4e66fb3158"
 					(reference "C18")
@@
 		)
 		(instances
-			(project "main_MagicAlonso__test"
+			(project "main_MagicAlonso"
 				(path "/80af5e1a-3060-4775-9fc3-f6762d1535e7/38d4c26b-5042-47e6-b450-9f4e66fb3158"
 					(reference "#PWR057")
@@
 		)
 		(instances
-			(project "main_MagicAlonso__test"
+			(project "main_MagicAlonso"
 				(path "/80af5e1a-3060-4775-9fc3-f6762d1535e7/38d4c26b-5042-47e6-b450-9f4e66fb3158"
 					(reference "C22")
@@
 		)
 		(instances
-			(project "main_MagicAlonso__test"
+			(project "main_MagicAlonso"
 				(path "/80af5e1a-3060-4775-9fc3-f6762d1535e7/38d4c26b-5042-47e6-b450-9f4e66fb3158"
 					(reference "#PWR059")
@@
 		)
 		(instances
-			(project "main_MagicAlonso__test"
+			(project "main_MagicAlonso"
 				(path "/80af5e1a-3060-4775-9fc3-f6762d1535e7/38d4c26b-5042-47e6-b450-9f4e66fb3158"
 					(reference "C19")
@@
 		)
 		(instances
-			(project "main_MagicAlonso__test"
+			(project "main_MagicAlonso"
 				(path "/80af5e1a-3060-4775-9fc3-f6762d1535e7/38d4c26b-5042-47e6-b450-9f4e66fb3158"
 					(reference "R17")
@@
 		)
 		(instances
-			(project "main_MagicAlonso__test"
+			(project ""
 				(path "/80af5e1a-3060-4775-9fc3-f6762d1535e7/38d4c26b-5042-47e6-b450-9f4e66fb3158"
 					(reference "L1")
@@
 		)
 		(instances
-			(project "main_MagicAlonso__test"
+			(project "main_MagicAlonso"
 				(path "/80af5e1a-3060-4775-9fc3-f6762d1535e7/38d4c26b-5042-47e6-b450-9f4e66fb3158"
 					(reference "Rp2")
@@
 		)
 		(instances
-			(project "main_MagicAlonso__test"
+			(project "main_MagicAlonso"
 				(path "/80af5e1a-3060-4775-9fc3-f6762d1535e7/38d4c26b-5042-47e6-b450-9f4e66fb3158"
 					(reference "#PWR061")
@@
 		)
 		(instances
-			(project "main_MagicAlonso__test"
+			(project "main_MagicAlonso"
 				(path "/80af5e1a-3060-4775-9fc3-f6762d1535e7/38d4c26b-5042-47e6-b450-9f4e66fb3158"
 					(reference "#PWR058")
@@
 		)
 		(instances
-			(project "main_MagicAlonso__test"
+			(project ""
 				(path "/80af5e1a-3060-4775-9fc3-f6762d1535e7/38d4c26b-5042-47e6-b450-9f4e66fb3158"
 					(reference "ST1")
@@
 		)
 		(instances
-			(project "main_MagicAlonso__test"
+			(project ""
 				(path "/80af5e1a-3060-4775-9fc3-f6762d1535e7/38d4c26b-5042-47e6-b450-9f4e66fb3158"
 					(reference "C17")
@@
 		)
 		(instances
-			(project "main_MagicAlonso__test"
+			(project ""
 				(path "/80af5e1a-3060-4775-9fc3-f6762d1535e7/38d4c26b-5042-47e6-b450-9f4e66fb3158"
 					(reference "U6")
@@
 		)
 		(instances
-			(project "main_MagicAlonso__test"
+			(project "main_MagicAlonso"
 				(path "/80af5e1a-3060-4775-9fc3-f6762d1535e7/38d4c26b-5042-47e6-b450-9f4e66fb3158"
 					(reference "#PWR062")
@@
 		)
 		(instances
-			(project "main_MagicAlonso__test"
+			(project "main_MagicAlonso"
 				(path "/80af5e1a-3060-4775-9fc3-f6762d1535e7/38d4c26b-5042-47e6-b450-9f4e66fb3158"
 					(reference "C21")
@@
 		)
 		(instances
-			(project "main_MagicAlonso__test"
+			(project "main_MagicAlonso"
 				(path "/80af5e1a-3060-4775-9fc3-f6762d1535e7/38d4c26b-5042-47e6-b450-9f4e66fb3158"
 					(reference "R16")
@@
 		)
 		(instances
-			(project "main_MagicAlonso__test"
+			(project ""
 				(path "/80af5e1a-3060-4775-9fc3-f6762d1535e7/38d4c26b-5042-47e6-b450-9f4e66fb3158"
 					(reference "RV1")
