File: pcb/main_Magic-simple/main_Magic-simple.kicad_pcb (KiCad board)
At the start: 2 copper layers, 89 x 113.2 mm, 53 parts, among them J1 PW, J10 ESC1, J11 ESC2, J12 ESC3, J14 UART_Out, J2 MPU6050, J3 LiPo-Battery, J9 Sensors, Q1 IRLML2502, SW2 EN_Push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

Commit message: simple main board added and donde
Parts:
- removed the ? at (97.7, 210.9)
- removed the ? at (106.5, 210.9)
- removed the ? at (115.3, 210.9)
- removed C1, C12, C5: 100nF, Capacitor_SMD:C_0805_2012Metric
- removed C11: 47uF, Capacitor_SMD:CP_Elec_6.3x5.4
- removed F1: 500mA, Fuse:Fuse_1812_4532Metric_Pad1.30x3.40mm_HandSolder
- removed J3: LiPo-Battery, TerminalBlock_Phoenix:TerminalBlock_Phoenix_PT-1,5-2-3.5-H_1x02_P3.50mm_Horizontal
- removed Q1: IRLML2502, Package_TO_SOT_SMD:SOT-23
- removed R10: 330, Resistor_SMD:R_0805_2012Metric
- removed R8: 10k, Resistor_SMD:R_0805_2012Metric
- added ?: , , F.Cu at (88.8, 174.9)
- added ?: , , F.Cu at (134.2, 160.8)
- added ?: , , F.Cu at (65.6, 178.7)
- added C28: 470uF, Capacitor_THT:CP_Radial_D8.0mm_P3.50mm, F.Cu at (135.1, 231.8)
- added C6: 100nF, Capacitor_SMD:C_0805_2012Metric, F.Cu at (137.2, 138.9)
- added D2: WS2812B, LED_SMD:LED_WS2812B_PLCC4_5.0x5.0mm_P3.2mm, F.Cu at (131.6, 136.3)
- added D4: LED_ON, MixLib:LED_0805_2012Metric, F.Cu at (64.5, 227.8)
- added H11: M3, MountingHole:MountingHole_3mm, F.Cu at (65.2, 234.8)
- added H12: M3, MountingHole:MountingHole_3mm, F.Cu at (147.8, 234.7)
- added J4: LiPo, Connector_JST:JST_XH_S2B-XH-A_1x02_P2.50mm_Horizontal, F.Cu at (128.0, 232.4)
- added JP1: ESP_JP, Resistor_SMD:R_1206_3216Metric, F.Cu at (63.1, 175.6)
- added JP2: LED_JP, Resistor_SMD:R_1206_3216Metric, F.Cu at (121.6, 142.9)
- added R1: 330, Resistor_SMD:R_0805_2012Metric, F.Cu at (140.4, 138.9)
- added R7: 4.7k, Resistor_SMD:R_0603_1608Metric, F.Cu at (64.5, 230.4)
- added SW1: Power_SW, Button_Switch_THT:SW_Push_2P2T_Toggle_CK_PVA2OAH5xxxxxxV2, F.Cu at (95.1, 228.8)
- C2: footprint Capacitor_SMD:CP_Elec_6.3x5.4 -> Capacitor_THT:CP_Radial_D8.0mm_P3.50mm
- J1: footprint Connector_JST:JST_XH_S2B-XH-A_1x02_P2.50mm_Horizontal -> Connector_JST:JST_XH_B2B-XH-A_1x02_P2.50mm_Vertical
- R4: value 20 -> 330; footprint Resistor_SMD:R_1206_3216Metric -> Resistor_SMD:R_0805_2012Metric
- SW2, SW3: footprint Button_Switch_SMD:SW_SPST_CK_RS282G05A3 -> MixLib:SW_Push_SPST_NO_Alps_SKRK_Handsolder
- U6: value Mini360 -> CN3903
- moved J10 231.2 mm to (113.0, 210.9)
- moved J11 224.2 mm to (105.3, 210.9)
- moved J1 223.9 mm to (143.8, 176.8), turned to 180 degrees
- moved C2 218.5 mm to (142.6, 227.4), turned to -90 degrees
- moved J12 218.4 mm to (97.5, 210.9)
- moved U6 216.0 mm to (77.8, 231.6), turned to 180 degrees
- moved D1 204.7 mm to (125.5, 226.8)
- moved BZ1 193.5 mm to (131.3, 177.1), turned to 90 degrees
- moved J14 168.5 mm to (144.4, 169.6), turned to 90 degrees
- moved J9 164.5 mm to (117.8, 134.2), turned to 180 degrees
- moved R4 162.8 mm to (133.2, 164.8)
- moved J2 155.7 mm to (137.6, 149.3), turned to -90 degrees
- moved C3 146.1 mm to (65.6, 175.0), turned to -90 degrees
- moved C4 143.6 mm to (67.7, 175.0), turned to -90 degrees
- moved R5 140.1 mm to (90.7, 135.9), turned to 90 degrees
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Connections:
- BZ1 pad 1: Net-(BZ1-+) -> /BUZ
- J14 pad 4: unconnected-(J14-Pin_4-Pad4) -> /VM
- J9 pad 9: Net-(J9-Pin_9) -> +3.3V
- R4 pad 1: Net-(BZ1-+) -> Net-(BZ1--)
- R4 pad 2: /Vb -> GND
- U1 pad 10: unconnected-(U1-IO25-Pad10) -> /ESC_1
- U1 pad 11: unconnected-(U1-IO26-Pad11) -> /BUZ
- U1 pad 12: unconnected-(U1-IO27-Pad12) -> /Data_2aux
- U1 pad 13: unconnected-(U1-IO14-Pad13) -> /LED_BLUE
- U1 pad 14: /ESC_1 -> /LED_RGB
- U1 pad 16: /ESC_2 -> /Data_1aux
- U1 pad 23: /ESC_3 -> /Data_SIG
- U1 pad 24: /LED_BLUE -> /Data_S3
- U1 pad 27: /Data_S3 -> /Data_S2
- U1 pad 28: /Data_S2 -> /Data_S1
- U1 pad 29: /LED_RGB -> unconnected-(U1-IO5-Pad29)
- U1 pad 30: /Data_S1 -> /Data_S0
- U1 pad 31: /Data_S0 -> /Data_EN
- U1 pad 37: /Data_EN -> /BUTTON
- U1 pad 4: /BUTTON -> /Enc1
- U1 pad 5: /Data_SIG -> /Enc2
- U1 pad 6: unconnected-(U1-IO34-Pad6) -> /CurrESC1&2
- U1 pad 7: /Data_1aux -> /CurrESC2
- U1 pad 8: /Data_2aux -> /ESC_3
- U1 pad 9: /BUZ -> /ESC_2
- U6 pad 3: unconnected-(U6-OUT-Pad3) -> +3.3V
Routing:
- net +3.3V: track 0.00 -> 265.0 mm, vias 0 -> 4
- net /RX: track 0.00 -> 114.1 mm, vias 0 -> 1
- net /TX: track 0.00 -> 109.6 mm, vias 0 -> 1
- net /Data_2aux: track 0.00 -> 96.9 mm
- net /VM: track 0.00 -> 95.1 mm
- net /SCL: track 0.00 -> 91.8 mm, vias 0 -> 1
- net /Data_1aux: track 0.00 -> 88.8 mm
- net /SDA: track 0.00 -> 87.7 mm, vias 0 -> 1
- net /BUZ: track 0.00 -> 62.6 mm, vias 0 -> 1
- net /ESC_1: track 0.00 -> 57.4 mm
- net /D_LED1: track 0.00 -> 55.3 mm, vias 0 -> 2
- net /ESC_2: track 0.00 -> 51.6 mm
- net /ESC_3: track 0.00 -> 48.9 mm
- net /EN: track 0.00 -> 43.8 mm, vias 0 -> 2
- net /LED_RGB: track 0.00 -> 42.9 mm, vias 0 -> 2
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Other:
- board size 89 x 113.2 mm -> 95.3 x 113.2 mm
