File: pcb/main_Alonso_JLC/main_Alonso_JLC.kicad_sch (KiCad schematic)
At the start: 0 parts

Commit message: pcb
Parts:
- added BZ1: Buzzer, Buzzer_Beeper:Buzzer_12x9.5RM7.6, symbol Device:Buzzer
- added C1, C11, C2, C5, C8, C9: 100nF, Capacitor_SMD:C_0603_1608Metric, symbol Device:C_Small
- added C10, C6, C7: 10uF, Capacitor_SMD:C_0805_2012Metric, symbol Device:C_Small
- added C3: 10UF, Capacitor_SMD:C_0805_2012Metric, symbol Device:C_Small
- added C4: 100nF, Capacitor_SMD:C_0805_2012Metric, symbol Device:C_Small
- added D1: SS14, Diode_SMD:D_SOD-123, symbol Device:D_Schottky_Small
- added D2: LED_RGB, LED_SMD:LED_RGB_5050-6, symbol Device:LED_RGB
- added D3, D4, D6: LED_BLUE, MixLib:LED_0805_2012Metric, symbol Device:LED_Small
- added H1, H11, H12, H2, H3, H4: M3, MountingHole:MountingHole_3mm, symbol Mechanical:MountingHole
- added H10, H7, H8, H9: M2, MountingHole:MountingHole_2.2mm_M2, symbol Mechanical:MountingHole
- added J2: MPU6050, MixLib:MPU6050_Module, symbol Connector:Conn_01x04_Pin
- added J5: ESC, Connector_JST:JST_XH_B6B-XH-A_1x06_P2.50mm_Vertical, symbol Connector:Conn_01x06_Pin
- added J9: Sensors, Connector_JST:JST_XH_S10B-XH-A_1x10_P2.50mm_Horizontal, symbol Connector:Conn_01x10_Pin
- added Q1: IRLML2502, Package_TO_SOT_SMD:SOT-23, symbol Transistor_FET:IRLML2060
- added R1, R13, R9: 10k, Resistor_SMD:R_0603_1608Metric, symbol Device:R_Small
- added R10, R11, R12, R2, R6, R7: 1k, Resistor_SMD:R_0603_1608Metric, symbol Device:R_Small
- added R14: 10k, Resistor_SMD:R_0805_2012Metric, symbol Device:R_Small
- added R16: 20k, Resistor_SMD:R_0805_2012Metric, symbol Device:R_Small
- added R3: 330k, Resistor_SMD:R_0805_2012Metric, symbol Device:R_Small
- added R4: 100k, Resistor_SMD:R_0805_2012Metric, symbol Device:R_Small
- added R5: 1k, Resistor_SMD:R_0805_2012Metric, symbol Device:R_Small
- added R8: 330, Resistor_SMD:R_0805_2012Metric, symbol Device:R_Small
- added SW1: Power_SW, MixLib:SW_DPDT_SLIDE_THT, symbol Switch:SW_Push_DPDT
- added SW2: PUSH_2, MixLib:SW_Push_Sw-3424p_Handsolder, symbol Switch:SW_Push
- added SW3: PUSH_3, MixLib:SW_Push_Sw-3424p_Handsolder, symbol Switch:SW_Push
- added SW4: PUSH_1, MixLib:SW_Push_Sw-3424p_Handsolder, symbol Switch:SW_Push
- added U1: STM32F103C8Tx, Package_QFP:LQFP-48_7x7mm_P0.5mm, symbol MCU_ST_STM32F1:STM32F103C8Tx
- added U2: AMS1117CD-3.3, Package_TO_SOT_SMD:TO-252-3_TabPin2, symbol Regulator_Linear:AMS1117CD-3.3
- added U2: BluePill_SWD_Breakout, MixLib:BluePill, symbol MixLib:BluePill_SWD_Breakout
- added U6: CN3905, MixLib:Mini360_step-down, symbol MixLib:Mini360
Connections:
- new net: D4.1 (K), R7.1
- new net: D2.5 (GA), R11.1
- new net: D3.1 (K), R2.1
- new net: R3.2, R4.1, R5.2
- new net: SW1.2 (B), SW1.5 (B), U6.1 (IN)
- new net: BZ1.2 (-), Q1.3 (D)
- new net: Q1.1 (G), R8.1
- new net: D6.1 (K), R6.1
- new net: D2.4 (BA), R10.1
- new net: D2.6 (RA), R12.1
- new net +3.3V: C10.1, C11.1, C2.1, C3.1, C4.1, C5.1, C7.1, C8.1, C9.1, J2.1 (Pin_1), J9.9 (Pin_9), SW2.1, SW3.1, SW4.1, U1.1 (VBAT), U1.24 (VDD), U1.36 (VDD), U1.48 (VDD), U1.9 (VDDA), U2.2 (VO), U2.20 (3V3), U2.38 (3V3)
- new net +5V: C1.1, C6.1, U2.3 (VI), U6.3 (OUT)
- new net BL_RX: U2.35 (PB10)
- new net BL_TX: U2.36 (PB11)
- new net BUZ: R8.2, U2.17 (PB9)
- new net Curr: R14.1
- new net Curr_3V3: R14.2, R16.1, U2.34 (PB1)
- new net Data_1aux: J9.2 (Pin_2), U2.25 (PA0)
- new net Data_2aux: J9.1 (Pin_1), U2.26 (PA1)
- new net Data_EN: J9.8 (Pin_8), U2.32 (PA7)
- new net Data_S0: J9.7 (Pin_7), U2.31 (PA6)
- new net Data_S1: J9.6 (Pin_6), U2.30 (PA5)
- new net Data_S2: J9.5 (Pin_5), U2.29 (PA4)
- new net Data_S3: J9.4 (Pin_4), U2.28 (PA3)
- new net Data_SIG: J9.3 (Pin_3), U2.27 (PA2)
- new net ESC_M1: U2.7 (PA10)
- new net ESC_M2: U2.6 (PA9)
- new net ESC_M3: U2.5 (PA8)
- new net GND: C1.2, C10.2, C11.2, C2.2, C3.2, C4.2, C5.2, C6.2, C7.2, C8.2, C9.2, D2.1 (RK), D2.2 (GK), D2.3 (BK), J2.2 (Pin_2), J9.10 (Pin_10), Q1.2 (S), R1.1, R13.1, R16.2, R2.2, R4.2, R6.2, R7.2, R9.1, U1.23 (VSS), U1.35 (VSS), U1.47 (VSS), U1.8 (VSSA), U2.1 (GND), U2.19 (GND), U2.39 (GND), U2.40 (GND), U6.2 (GND)
- new net LED_G: D6.2 (A), U2.12 (PB4)
- new net LED_O: D3.2 (A), U2.13 (PB5)
- new net LED_R: D4.2 (A), U2.16 (PB8)
- new net PUSH_1: R9.2, SW4.2, U2.24 (PC15)
- new net PUSH_2: R1.2, SW2.2, U2.23 (PC14)
- new net PUSH_3: R13.2, SW3.2, U2.22 (PC13)
- new net RGB_B: R10.2, U2.2 (PB13)
- new net RGB_G: R11.2, U2.3 (PB14)
- new net RGB_R: R12.2, U2.4 (PB15)
- new net RST: U2.37 (RST)
- new net SCL: J2.3 (Pin_3), U2.14 (PB6)
- new net SDA: J2.4 (Pin_4), U2.15 (PB7)
- new net VM: D1.2 (A), R3.1
- new net V_LiPo: R5.1
- new net V_bat: U2.33 (PB0)
- new net Vb: BZ1.1 (+), D1.1 (K), SW1.1 (A), SW1.4 (A)
- no-connect marks 0 -> 8
Other:
- note added: "Battery Supply"
- note added: "Battery level"
- note added: "Button"
- note added: "ESCs Connections"
- note added: "I2C Connections"
- note added: "Interfaces"
- note added: "MCU"
- note added: "Mounting Holes"
- note added: "Passive Buzzer"
- note added: "RGB LED"
- note added: "Sensors Input"

Commit message: jlc pcb schematic
Parts:
- removed BZ1: Buzzer, Buzzer_Beeper:Buzzer_12x9.5RM7.6, symbol Device:Buzzer
- removed J5: ESC, Connector_JST:JST_XH_B6B-XH-A_1x06_P2.50mm_Vertical, symbol Connector:Conn_01x06_Pin
- removed Q1: IRLML2502, Package_TO_SOT_SMD:SOT-23, symbol Transistor_FET:IRLML2060
- added C12, C17, C22, C25: 100nF, Capacitor_SMD:C_0603_1608Metric, symbol Device:C_Small
- added C13, C14, C15, C16: 20pF, Capacitor_SMD:C_0603_1608Metric, symbol Device:C_Small
- added C18, C19, C20, C21: 1uF, Capacitor_SMD:C_0805_2012Metric, symbol Device:C_Small
- added C23: 2.2nF, Capacitor_SMD:C_0603_1608Metric, symbol Device:C_Small
- added C26: 1uF, Capacitor_SMD:C_0603_1608Metric, symbol Device:C_Small
- added D5: LED_ON, MixLib:LED_0805_2012Metric, symbol Device:LED_Small
- added R15: 10k, Resistor_SMD:R_0603_1608Metric, symbol Device:R_Small
- added R17: 1k, Resistor_SMD:R_0603_1608Metric, symbol Device:R_Small
- added R18: 4.7k, Resistor_SMD:R_0603_1608Metric, symbol Device:R_Small
- added SW5: PUSH_3, MixLib:SW_Push_Sw-3424p_Handsolder, symbol Switch:SW_Push
- added SW6: BOOT_SW, symbol Switch:SW_SPDT
- added U3: MPU-6050, Sensor_Motion:InvenSense_QFN-24_4x4mm_P0.5mm, symbol Sensor_Motion:MPU-6050
- added Y1: 8MHz, Crystal:Crystal_SMD_5032-4Pin_5.0x3.2mm, symbol Device:Crystal_GND24_Small
- added Y2: 32.768KHz, Crystal:Crystal_SMD_Abracon_ABS25-4Pin_8.0x3.8mm, symbol Device:Crystal_GND23_Small
- C10: value 10uF -> 1uF
- D3: value LED_BLUE -> LED_ORANGE
- D4: value LED_BLUE -> LED_RED
- D6: value LED_BLUE -> LED_GREEN
- R14: value 10k -> 1M; footprint Resistor_SMD:R_0805_2012Metric -> Resistor_SMD:R_0603_1608Metric
- R16: value 20k -> 10k; footprint Resistor_SMD:R_0805_2012Metric -> Resistor_SMD:R_0603_1608Metric
- R8: value 330 -> 10k; footprint Resistor_SMD:R_0805_2012Metric -> Resistor_SMD:R_0603_1608Metric
Connections:
- net +3.3V: now also D2.4 (BA), D2.5 (GA), D2.6 (RA), D3.2 (A), D4.2 (A), D6.2 (A), R8.2, C17.1, C18.1, C19.1, C20.1, C21.1, C25.1, C26.1, D5.2 (A), R18.2, SW6.3 (C), U3.13 (VDD), U3.8 (VLOGIC)
- net BL_RX: now also U1.12 (PA2)
- net BL_TX: now also U1.13 (PA3)
- net BUZ: no longer R8.2
- net Curr: no longer R14.1
- net Curr_3V3: no longer R14.2, R16.1
- net GND: now also R16.1, C12.2, C13.2, C14.2, C15.2, C16.2, C17.2, C18.2, C19.2, C20.2, C21.2, C22.2, C23.2, C25.2, C26.2, R17.2, SW5.2, SW6.1 (A), U3.1 (CLKIN), U3.18 (GND), U3.9 (AD0), Y1.2, Y1.4, Y2.2, Y2.3; no longer D2.1 (RK), D2.2 (GK), D2.3 (BK), R16.2, R2.2, R6.2, R7.2
- net LED_G: now also R6.2; no longer D6.2 (A)
- net LED_O: now also R2.2; no longer D3.2 (A)
- net LED_R: now also R7.2; no longer D4.2 (A)
- net at R11.1: now also D2.2 (GK); no longer D2.5 (GA)
- net NRST: now reaches R8.1
- net NRST: now also U1.7 (NRST), C12.1, SW5.1
- net at U1.20 (PB2): now also R16.2
- net RCC_IN: now reaches U1.3 (PC14)
- net RCC_IN: now also C15.1, Y2.1
- net CH340C_RX: now reaches U1.30 (PA9)
- net CH340C_TX: now reaches U1.31 (PA10)
- net RCC_OUT: now reaches U1.4 (PC15)
- net RCC_OUT: now also C16.1, Y2.4
- net at U1.44 (BOOT0): now also R15.2
- net OSC_IN: now reaches U1.5 (PD0)
- net OSC_IN: now also R14.2, C13.1, Y1.1
- net OSC_OUT: now reaches U1.6 (PD1)
- net OSC_OUT: now also R14.1, C14.1, Y1.3
- net at R10.1: now also D2.3 (BK); no longer D2.4 (BA)
- net at R12.1: now also D2.1 (RK); no longer D2.6 (RA)
- new net: R15.1, SW6.2 (B)
- new net: D5.1 (K), R17.1
- new net: C23.1, U3.20 (CPOUT)
- new net: C22.1, U3.10 (REGOUT)
- new net INT_MPU: U3.12 (INT)
- new net MPU_SCL: U3.23 (SCL)
- new net MPU_SDA: R18.1, U3.24 (SDA)
- no-connect marks 8 -> 12
Other:
- note added: "MPU6050"
- note added: "Power Supply"
- note removed: "Battery Supply"
- note removed: "Battery level"
- note removed: "Button"
- note removed: "ESCs Connections"
- note removed: "I2C Connections"
- note removed: "Interfaces"
- note removed: "Passive Buzzer"
- note removed: "RGB LED"
- note removed: "Sensors Input"
- moved on the sheet: C1, C10, C11, C2, C5, C6, C7, C8, C9, D1, D2, J2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

Commit message: pcb
Parts:
- removed C3: 10UF, Capacitor_SMD:C_0805_2012Metric, symbol Device:C_Small
- removed C4: 100nF, Capacitor_SMD:C_0805_2012Metric, symbol Device:C_Small
- removed D4: LED_RED, MixLib:LED_0805_2012Metric, symbol Device:LED_Small
- removed H1, H2, H3, H4: M3, MountingHole:MountingHole_3mm, symbol Mechanical:MountingHole
- removed H7: M2, MountingHole:MountingHole_2.2mm_M2, symbol Mechanical:MountingHole
- removed J2: MPU6050, MixLib:MPU6050_Module, symbol Connector:Conn_01x04_Pin
- removed R5: 1k, Resistor_SMD:R_0805_2012Metric, symbol Device:R_Small
- removed R7: 1k, Resistor_SMD:R_0603_1608Metric, symbol Device:R_Small
- removed U2: BluePill_SWD_Breakout, MixLib:BluePill, symbol MixLib:BluePill_SWD_Breakout
- removed U6: CN3905, MixLib:Mini360_step-down, symbol MixLib:Mini360
- added C1: 1uF, Capacitor_SMD:C_0805_2012Metric, symbol Device:C_Small
- added C6: 100nF, Capacitor_SMD:C_0603_1608Metric, symbol Device:C_Small
- added C7: 1uF, Capacitor_SMD:C_0603_1608Metric, symbol Device:C_Small
- added H6: M2, MountingHole:MountingHole_2.2mm_M2, symbol Mechanical:MountingHole
- added J1: ESC, MixLib:pad_smd_x5, symbol Connector:Conn_01x06_Pin
- added J3: SWD, Connector_JST:JST_XH_B4B-XH-A_1x04_P2.50mm_Vertical, symbol Connector:Conn_01x04_Pin
- added J5: HC05, MixLib:HC05, symbol Connector:Conn_01x04_Pin
- added J7: XT30, Connector_AMASS:AMASS_XT30U-F_1x02_P5.0mm_Vertical, symbol MixLib:XT30PW-M
- added JP1: BL_PW, Jumper:SolderJumper-3_P1.3mm_Bridged123_RoundedPad1.0x1.5mm, symbol Jumper:SolderJumper_3_Bridged12
- added R15: >20k, Resistor_SMD:R_0805_2012Metric, symbol Device:R_Small
- added R17: 4.7k, Resistor_SMD:R_0603_1608Metric, symbol Device:R_Small
- added TP4: GND, TestPoint:TestPoint_Pad_D1.5mm, symbol PCM_4ms_Connector:TestPoint
- added TP5: 3V3, TestPoint:TestPoint_Pad_D1.5mm, symbol PCM_4ms_Connector:TestPoint
- added U1: TL071HIDBV, PCM_Package_TO_SOT_SMD_AKL:SOT-23-5, symbol PCM_Amplifier_Operational_AKL:TL071HIDBV
- added U3: VL1838, MixLib:TL1838, symbol MixLib:TL1838
- D1: renamed from D6; value LED_GREEN -> LED_1
- D2: renamed from D3; value LED_ORANGE -> LED_2
- H11, H12: value M3 -> M2; footprint MountingHole:MountingHole_3mm -> MountingHole:MountingHole_2.2mm_M2
- SW5: renamed from SW6; footprint (none) -> MixLib:SW_DPDT_SLIDE_THT
- renumbered C22 to C10, C23 to C11, C21 to C12, C19 to C13, C12 to C14, C20 to C15, C13 to C16, C18 to C17, C10 to C18, C14 to C19, C6 to C2, C2 to C20, C8 to C21, C15 to C22, C9 to C23, C11 to C24, C16 to C25, C17 to C26, C1 to C3, C5 to C4, C7 to C5, C26 to C8, C25 to C9, D2 to D7, D1 to D8, D5 to D9, H9 to H5, H10 to H9, J9 to J4, R6 to R1, R11 to R10, R12 to R11, R13 to R12, R3 to R13, R4 to R14, R17 to R16, R8 to R19, R16 to R20, R15 to R21, R14 to R22, R9 to R7, R1 to R8, R10 to R9, SW4 to SW1, SW1 to SW4, SW5 to SW6, U3 to U4, U1 to U5
Connections:
- net LED_G is gone; now on net LED_1: R1.2
- net LED_O is gone; now on net LED_2: R2.2
- net +3.3V: now also C1.2, C6.1, C7.1, J3.4 (Pin_4), JP1.3 (B), R15.1, R17.2, TP5.1, U3.3 (VCC)
- net +5V: now also JP1.2 (C)
- net BL_RX: now also U5.21 (PB10), J5.1 (Pin_1); no longer U5.12 (PA2)
- net BL_TX: now also U5.22 (PB11), J5.2 (Pin_2); no longer U5.13 (PA3)
- net Curr: now also U5.19 (PB1), J1.6 (Pin_6)
- net Data_1aux: now also U5.16 (PA6)
- net Data_2aux: now also U5.17 (PA7)
- net Data_EN: now also U5.10 (PA0)
- net Data_S0: now also U5.11 (PA1)
- net Data_S1: now also U5.12 (PA2)
- net Data_S2: now also U5.13 (PA3)
- net Data_S3: now also U5.14 (PA4)
- net Data_SIG: now also U5.15 (PA5)
- net ESC_M1: now also U5.42 (PB6), J1.2 (Pin_2)
- net ESC_M2: now also U5.41 (PB5), J1.3 (Pin_3)
- net ESC_M3: now also U5.40 (PB4), J1.4 (Pin_4)
- net ESC_M4: now also U5.39 (PB3), J1.5 (Pin_5)
- net GND: now also C1.1, C6.2, C7.2, J1.1 (Pin_1), J3.1 (Pin_1), J5.3 (Pin_3), J7.N, R15.2, TP4.1, U3.2 (GND)
- net MPU_SCL: now also U5.45 (PB8), R17.1
- net MPU_SDA: now also U5.46 (PB9)
- net PUSH_1: now also U5.25 (PB12)
- net PUSH_2: now also U5.26 (PB13)
- net PUSH_3: now also U5.27 (PB14)
- net RGB_B: now also U5.29 (PA8)
- net RGB_G: now also U5.32 (PA11)
- net RGB_R: now also U5.33 (PA12)
- net VM: now also J7.P
- net V_LiPo: now also U5.18 (PB0), U1.1, U1.4 (-)
- net at R13.2, R14.1: now also U1.3 (+)
- net CN3903/Vin: now reaches SW4.2 (B), SW4.5 (B)
- net LED_2: now reaches U5.28 (PB15)
- net SWDIO: now reaches U5.34 (PA13)
- net SWDIO: now also J3.3 (Pin_3)
- net SWCLK: now reaches U5.37 (PA14)
- net SWCLK: now also J3.2 (Pin_2)
- net LED_1: now reaches U5.38 (PA15)
- net IR: now reaches U5.43 (PB7)
- net IR: now also U3.1 (OUT)
- new net: J5.4 (Pin_4), JP1.1 (A)
- no-connect marks 12 -> 8
Other:
- added sheet CH340C (CH340G_programmer.kicad_sch)
- added sheet CN3903 (CN3903-StepDown.kicad_sch)
- added sheet Encoders_PCB (Encoders_PCB.kicad_sch)
- note added: "*R19 es opcional según datasheet."
- note added: "Bluetooth"
- note added: "Buttons"
- note added: "Encoders"
- note added: "Holes"
- note added: "IR Receiver"
- note added: "LEDs"
- note added: "LiPo Voltage"
- note added: "Power Input"
- note added: "Power Regulation"
- note added: "Programming"
- note added: "Sensors input"
- note added: "TODO: ordenar"
- note removed: "MCU"
- note removed: "Mounting Holes"
- note removed: "Power Supply"
- moved on the sheet: C10, C11, C12, C13, C14, C15, C16, C17, C18, C19, C2, C20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
