File: pcb/main_Magic_BluePIll/main_Magic_BluePIll.kicad_sch (KiCad schematic)
At the start: 49 parts, among them J2 MPU6050, J5 ESC, J9 Sensors, Q1 IRLML2502, SW1 Power_SW, SW2 PUSH_2, SW3 PUSH_3, SW4 PUSH_1, U1 BluePill_SWD_Breakout, U2 AMS1117CD-3.3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

Commit message: PID calibration & broken menu
Other:
- note added: "^ pd: rx y tx estan mal"
Changed lines of the file:
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@@
+		)
+	)
+	(text "^\npd: \nrx y tx\nestan mal\n"
+		(exclude_from_sim no)
+		(at 153.162 94.996 0)
+		(effects
+			(font
+				(size 0.65 0.65)
+				(thickness 0.25)
+				(italic yes)
+			)
 		)
 	)
